File: SpecialistEE20.brd (EAGLE design)
At the start: 52 parts

Commit message: +ee
Parts:
- added DD54: К580ВА86, ic-package:DIL20
- added DD55, DD56: К580ИР82, ic-package:DIL20
Changed lines of the file:
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@@
 <board>
 <plain>
-<dimension x1="13.97" y1="35.56" x2="180.34" y2="33.02" x3="97.155" y3="207.01" textsize="1.778" layer="21" dtype="horizontal"/>
-<dimension x1="-11.43" y1="135.89" x2="12.7" y2="38.1" x3="200.66" y3="86.995" textsize="1.778" layer="21" dtype="vertical"/>
-<text x="-22.86" y="149.86" size="6.4516" layer="22">21x13</text>
+<dimension x1="13.97" y1="35.56" x2="180.34" y2="33.02" x3="97.155" y3="194.31" textsize="1.778" layer="21" dtype="horizontal"/>
+<dimension x1="11.43" y1="133.35" x2="12.7" y2="38.1" x3="190.5" y3="85.725" textsize="1.778" layer="21" dtype="vertical"/>
+<text x="-19.05" y="152.4" size="6.4516" layer="22">21x13</text>
 </plain>
 <attributes>
@@
 <element name="DD47" library="74xx-eu" package="DIL14" value="К155ИР1" x="22.86" y="73.66" rot="R270"/>
 <element name="DD48" library="74xx-eu" package="DIL14" value="К155ИР1" x="36.83" y="72.39" rot="R270"/>
+<element name="DD54" library="ic-package" package="DIL20" value="К580ВА86" x="-6.35" y="26.67"/>
+<element name="DD55" library="ic-package" package="DIL20" value="К580ИР82" x="-6.35" y="13.97"/>
+<element name="DD56" library="ic-package" package="DIL20" value="К580ИР82" x="-6.35" y="1.27"/>
 </elements>
 <signals>

Commit message: .
Parts:
- removed DD13, DD14, DD51: К155ИД4, 74xx-eu:DIL14
- removed DD32, DD33, DD35, DD41, DD42: К565РУ3, ic-package:DIL16
- removed DD43: КР580ВМ80, micro-intel:DIL40
- removed DD44: КР580ВВ55, micro-intel:DIL40
- removed DD45: К155ЛН1, 74xx-eu:DIL14
- removed DD46: К589ИР12, ic-package:DIL24-6
- removed DD52: К573РФ2, memory:DIL24
- added C1: 300, rcl:C0805
- added DD19-: К155ЛИ1, 74xx-eu:DIL14
- added DD9-: К155ЛЕ1, 74xx-eu:DIL14
- added R1, R2: 390, rcl:M1206
- added U$1: (no value), simvol-ik:PCB-MAIN
- added Z1: 8000, crystal:HC49/S
- DD19: value К155ЛИ1 -> 74LS365N; device 74xx-eu:DIL14 -> 74xx-eu:DIL16
- DD21, DD22, DD23, DD24, DD25, DD26, DD27, DD28: value К565РУ3 -> КР565РУ5
- DD29: value К565РУ3 -> КР580ВМ80; device ic-package:DIL16 -> micro-intel:DIL40
- DD30: value К565РУ3 -> КР580ВВ55; device ic-package:DIL16 -> micro-intel:DIL40
- DD31: value К565РУ3 -> К589ИР12; device ic-package:DIL16 -> ic-package:DIL24-6
- DD34: value К565РУ3 -> К555АП6; device ic-package:DIL16 -> 74xx-eu:DIL20
- DD36: value К565РУ3 -> К155ИД4; device ic-package:DIL16 -> 74xx-eu:DIL14
- DD37, DD38: value К565РУ3 -> К573РФ2; device ic-package:DIL16 -> memory:DIL24
- DD39: value К565РУ3 -> (none); device ic-package:DIL16 -> memory:DIL28
- DD40: value К565РУ3 -> К155ИД4; device ic-package:DIL16 -> 74xx-eu:DIL16
- DD9: value К155ЛЕ1 -> К155ЛН1
- moved DD30 148.4 mm to (213.4, 97.8), turned to 90 degrees
- moved DD8 145.6 mm to (31.8, 144.8), turned to 0 degrees
- moved DD7 142.9 mm to (30.5, 86.4), turned to 0 degrees
- moved DD40 142.8 mm to (31.8, 128.3), turned to 0 degrees
- moved DD37 134.6 mm to (156.2, 72.4), turned to 0 degrees
- moved DD36 128.2 mm to (123.2, 52.1), turned to 0 degrees
- moved DD11 125.1 mm to (30.5, 71.1), turned to 0 degrees
- moved DD38 121.9 mm to (156.2, 49.5), turned to 0 degrees
- moved DD5 119.6 mm to (54.6, 69.8), turned to 0 degrees
- moved DD50 117.1 mm to (138.4, 3.81)
- moved DD20 117.0 mm to (55.9, 128.3), turned to 0 degrees
- moved DD6 115.5 mm to (30.5, 114.3), turned to 0 degrees
- moved DD1 109.5 mm to (30.5, 158.8), turned to 0 degrees
- moved DD49 109.2 mm to (119.4, 8.89)
- moved DD25 106.4 mm to (123.2, 153.7)
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Connections:
- new net N$1: DD3.11, DD4.14
- new net N$11: DD2.5, DD8.12
- new net N$12: DD5.1, DD5.12
- new net N$13: DD4.1, DD4.12
- new net N$14: DD4.3, DD5.3, DD5.9
- new net N$16: DD4.2, DD5.2
- new net N$19: DD1.14, DD2.16, DD3.5, DD4.5, DD5.5
- new net N$2: DD4.11, DD5.14
- new net N$3: DD1.13, R1.1, Z1.1
- new net N$4: DD2.7, DD3.14
- new net N$5: C1.1, DD1.12, R1.2
- new net N$6: DD1.10, DD1.9, R2.2, Z1.2
- new net N$7: C1.2, DD1.11, R2.1
- new net N$8: DD1.8, DD8.5, DD9.13
- net GND: now also DD19-.7, DD19.8, DD2.14, DD3.2, DD3.3, DD30.7, DD34.10, DD36.7, DD37.12, DD38.12, DD39.14, DD40.8, DD8.14, DD9-.7; no longer DD13.7, DD14.7, DD19.7, DD44.7, DD45.7, DD51.7, DD52.12
- net VBB/-5V: now also DD29.11; no longer DD43.11
- net VCC: now also DD19-.14, DD19.16, DD30.26, DD34.20, DD36.14, DD37.24, DD38.24, DD39.28, DD40.16, DD9-.14; no longer DD1.14, DD13.14, DD14.14, DD19.14, DD2.16, DD3.5, DD4.5, DD44.26, DD45.14, DD5.5, DD51.14, DD52.24
- net VCC/+5V: now also DD29.20; no longer DD43.20
- net VDD/+12V: now also DD29.28; no longer DD43.28
- net VSS/GND: now also DD29.2; no longer DD43.2
Other:
- board text added: "220х135 вост экс нов"

Commit message: ..
Parts:
- added C3: 2m2, rcl:E2,5-5
- added C4, C4': (no value), rcl:C1206
- added JP1: (no value), Разъёмы штырьковые 2.54мм:1X01
- added R13: 2k, rcl:M1206
- added R3: 200, rcl:M1206
- added R4: 150, rcl:M1206
- added R47, R48: 390r 0.5w, rcl:0411/15
- added R5: 430*, rcl:M1206
- added R6: 390r, rcl:0411/15
- added VD1, VD10, VD2, VD3, VD3*, VD4, VD5, VD6, VD7, VD9: (no value), diode:SOD80C
- DD36: device 74xx-eu:DIL14 -> 74xx-eu:DIL16
- moved U$1 227.3 mm to (529.6, 193.0), turned to 180 degrees
- moved DD29 8.52 mm to (104.1, 110.5)
- moved DD9 7.73 mm to (55.9, 152.4)
- moved DD20 3.81 mm to (55.9, 132.1)
- moved DD36 3.59 mm to (125.7, 54.6)
Connections:
- net N$12 renamed G14
- net N$2 renamed G13
- new net +12V: R47.2, R48.2, R6.2
- new net +5V: R13.2, R5.2
- new net -5V: C4'.1, C4.1, VD2.A, VD3*.A, VD3.A
- new net CPU_F1: R47.1
- new net CPU_F2: R48.1
- new net G1: DD8.7
- new net G10: DD4.1, DD4.12, DD6.3
- new net G11: DD10.1, DD10.2, DD4.9
- new net G12: DD4.8, DD6.2
- new net G15: DD40.3, DD8.2
- new net G16: DD10.11, DD10.12, DD4.3, DD5.3, DD5.9, DD6.12
- new net G2: DD2.3
- new net G3: DD11.12, DD2.2
- new net G4: DD2.6, DD6.8
- new net G5: DD2.7, DD20.4, DD20.5, DD3.14, DD6.6
- new net G6: DD3.12, DD6.5
- new net G7: DD10.3, DD3.9
- new net G8: DD10.4, DD3.8
- new net G9: DD10.5, DD3.11, DD4.14
- new net N$10: DD36.6, VD5.C
- new net N$12: DD10.6, DD6.1
- new net N$15: DD36.11, VD6.C
- new net N$17: DD36.12, VD7.C
- new net N$18: R13.1, VD4.A, VD5.A, VD6.A, VD7.A
- new net N$2: DD1.5, DD6.11, DD6.4
- new net N$20: DD40.13, DD8.3
- new net N$21: C3.+, DD20.6, R6.1
- new net N$22: C3.-, VD1.A, VD2.C
- new net N$23: DD40.1, DD8.6
- new net N$24: DD40.2
- new net N$25: DD10.8, VD10.C
- new net N$26: DD11.11, DD3.1, VD9.C
- new net N$27: R3.2, R4.1, R5.1, VD10.A, VD9.A
- new net N$28: JP1.1, R4.2
- new net N$9: DD36.7, VD4.C
- net GND: now also C4'.2, C4.2, DD36.8, DD40.14, DD40.15, R3.1, VD1.C, VD3*.C, VD3.C; no longer DD36.7
- net N$1: now also DD11.13, DD6.10; no longer DD3.11, DD4.14
- net N$13: now also DD1.6, DD6.9; no longer DD4.1, DD4.12
- net N$14: now also DD1.3, DD6.13; no longer DD4.3, DD5.3, DD5.9
- net N$4: now also DD7.12, DD9-.3; no longer DD2.7, DD3.14
- net VCC: now also DD36.16; no longer DD36.14

Commit message: .
Parts:
- removed DD19-: К155ЛИ1, 74xx-eu:DIL14
- removed DD9-: К155ЛЕ1, 74xx-eu:DIL14
- added VD8: 1N4004, diode:DO41-10
- moved DD20 1.27 mm to (57.1, 132.1)
- renumbered DD54 to DD54.1, DD55 to DD55.1, DD56 to DD56.1
Connections:
- new net N$30: DD20.12, DD40.10
- new net N$31: DD20.8, DD20.9, DD40.12, DD7.10, DD7.11
- net +12V: now also VD8.C
- net +5V: now also DD1.14, DD10.14, DD11.14, DD12.14, DD2.16, DD3.5, DD4.5, DD5.5, DD6.14, DD7.14, DD8.16, DD9.14, VD8.A
- net CPU_F1: now also DD20.10, R48.1; no longer R47.1
- net CPU_F2: now also DD20.13, R47.1; no longer R48.1
- net G5: now also DD20.6; no longer DD20.4
- net GND: no longer DD19-.7, DD9-.7
- net N$19: now also DD20.11, DD40.9, DD7.9; no longer DD1.14, DD2.16, DD3.5, DD4.5, DD5.5
- net N$21: now also DD20.4; no longer DD20.6
- net N$24: now also DD1.4
- net N$4: now also DD40.4, DD9.3; no longer DD7.12, DD9-.3
- net VCC: no longer DD10.14, DD11.14, DD12.14, DD19-.14, DD6.14, DD7.14, DD8.16, DD9-.14, DD9.14

Commit message: ii
Parts:
- removed DD47, DD48: К155ИР1, 74xx-eu:DIL14
- removed DD49, DD50: К589АП16, ic-package:DIL16
- added DD101, DD102, DD103, DD104: КР565РУ5, ic-package:DIL16
- added DD105, DD108: К555ИР22, 74xx-eu:DIL20
- added DD106, DD109, DD32, DD33: К555ИР16, 74xx-eu:DIL14
- added DD107, DD110: К155ЛЕ1, 74xx-eu:DIL14
- added DD111, DD112: КР580ВВ55, micro-intel:DIL40
- added DD113, DD114: MEGA8-AI, atmel:TQFP32-08
- added DD113P: MEGA8-P, atmel:DIL28-3
- added DD14: К155ЛА3, 74xx-eu:DIL14
- added DD49.2, DD50.2: К589АП16, ic-package:DIL16
- DD19: value 74LS365N -> К155ЛП10
- moved DD54.1 252.0 mm to (208.3, 12.7)
- moved DD55.1 252.0 mm to (209.6, -2.54)
- moved DD56.1 252.0 mm to (209.6, -14.0)
- moved JP1 242.2 mm to (194.3, 214.6), turned to 180 degrees
- moved VD9 241.4 mm to (209.6, 198.1), turned to 90 degrees
- moved U$1 241.4 mm to (340.4, 43.2), turned to 0 degrees
- moved VD10 233.5 mm to (204.5, 198.1), turned to 90 degrees
- moved R3 225.8 mm to (199.4, 198.1), turned to 90 degrees
- moved R5 216.5 mm to (193.0, 198.1), turned to 90 degrees
- moved R47 207.5 mm to (186.7, 48.3), turned to 270 degrees
- moved R4 202.2 mm to (184.2, 196.8), turned to 90 degrees
- moved R1 199.9 mm to (204.5, 78.7), turned to 0 degrees
- moved R48 198.9 mm to (180.3, 48.3), turned to 270 degrees
- moved DD11 198.4 mm to (199.4, 175.3), turned to 180 degrees
- moved Z1 195.8 mm to (199.4, 73.7), turned to 180 degrees
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Connections:
- new net AVCC: DD113.18, DD113P.20, DD114.18
- net GND: now also DD105.10, DD106.7, DD107.7, DD108.10, DD109.7, DD110.7, DD111.7, DD112.7, DD113.21, DD113.3, DD113.5, DD113P.22, DD113P.8, DD114.21, DD114.3, DD114.5, DD14.7, DD32.7, DD33.7; no longer DD47.7, DD48.7
- net VCC: now also DD105.20, DD106.14, DD107.14, DD108.20, DD109.14, DD110.14, DD111.26, DD112.26, DD113.4, DD113.6, DD113P.7, DD114.4, DD114.6, DD14.14, DD32.14, DD33.14; no longer DD47.14, DD48.14

Commit message: .
Parts:
- added C10: 2m2, rcl:E2,5-5
- added C11: 22n, rcl:C0805
- added C5: 100, rcl:C0805
- added C6: 68, rcl:C0805
- added C7: 100m, rcl:E2,5-5
- added R10, R11: 2k, rcl:M1206
- moved VD8 180.5 mm to (227.3, 49.5), turned to 90 degrees
- moved DD49.2 177.6 mm to (270.5, 146.1)
- moved DD50.2 177.6 mm to (285.8, 146.1)
- moved DD54.1 177.6 mm to (311.1, 157.5)
- moved DD55.1 177.6 mm to (312.4, 142.2)
- moved DD56.1 177.6 mm to (312.4, 130.8)
- moved VD9 47.1 mm to (188.0, 156.2)
- moved VD10 36.4 mm to (189.2, 165.1)
- moved DD113 20.3 mm to (-15.2, 143.5)
- moved DD28 17.8 mm to (82.5, 92.7)
- moved DD27 15.2 mm to (94.0, 92.7)
- moved DD26 12.7 mm to (105.4, 92.7)
- moved DD25 10.2 mm to (116.8, 92.7)
- moved DD24 7.62 mm to (128.3, 92.7)
- moved DD23 5.08 mm to (139.7, 92.7)
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Connections:
- new net G17: DD11.9, DD20.12, DD40.10
- new net G18: C5.1, DD12.11, DD20.8, DD20.9, DD40.12, DD7.10, DD7.11
- new net G19: DD12.8
- new net K20: C7.+, DD12.2, R10.1
- new net N$29: DD2.1, DD2.10, DD2.15, DD2.9
- new net N$32: DD8.1, DD8.10, DD8.15, DD8.9
- new net N$33: C10.-, C11.2, JP1.1
- new net N$34: DD11.8, DD12.3
- new net N$36: DD12.12
- new net N$37: DD7.12, DD9.1
- net +5V: now also R10.2, R11.2
- net G10: now also DD7.2
- net G11: now also DD7.1
- net G12: now also DD7.13
- net G15: now also C6.1, DD1.1
- net G16: now also DD11.10
- net GND: now also C5.2, C6.2, C7.-
- net N$16: now also DD9.2
- net N$28: now also C10.+, C11.1; no longer JP1.1
- net N$30: now also DD1.2; no longer DD20.12, DD40.10
- net N$31: now also DD12.1, DD12.10, DD12.13, DD12.4, R11.1; no longer DD20.8, DD20.9, DD40.12, DD7.10, DD7.11

Commit message: ..
Parts:
- added RD1, RD2: 2k, rcl:M1206
- moved U$1 98.0 mm to (433.1, 74.9)
- moved DD101 11.4 mm to (-22.9, 90.2)
- moved DD103 7.62 mm to (-34.3, 90.2)
- moved DD102 3.81 mm to (-45.7, 90.2)
Connections:
- removed net N$32: DD8.1, DD8.10, DD8.15, DD8.9
- new net A'11: DD16.11
- new net A'12: DD17.5
- new net A'13: DD17.11
- new net A'14: DD18.10
- new net A'15: DD18.11
- new net A0: DD18.5
- new net A1: DD15.6
- new net A10: DD16.5
- new net A2: DD15.10
- new net A3: DD16.6
- new net A4: DD16.10
- new net A5: DD17.6
- new net A6: DD17.10
- new net A7: DD18.6
- new net A8: DD15.5
- new net A9: DD15.11
- new net MA0: DD15.7
- new net MA1: DD15.9
- new net MA2: DD16.7
- new net MA3: DD16.9
- new net MA4: DD17.7
- new net MA5: DD17.9
- new net MA6: DD18.7
- new net MA7: DD18.9
- new net N$38: DD8.1, DD8.10, DD8.11, DD8.15, DD8.4, DD8.9, RD2.2
- new net N$41: DD15.14, DD16.14, DD17.14, DD18.14
- net +5V: now also DD14.14, DD15.16, DD16.16, DD17.16, DD18.16, DD19.16, DD20.14, RD1.2, RD2.1
- net G1: now also DD15.3
- net G10: now also DD16.4
- net G11: now also DD16.12
- net G12: now also DD17.4
- net G13: now also DD17.12
- net G14: now also DD18.4
- net G19: now also DD15.2, DD16.2, DD17.2, DD18.2
- net G2: now also DD15.13
- net G3: now also DD16.3
- net G4: now also DD16.13
- net G5: now also DD17.3
- net G6: now also DD17.13
- net G7: now also DD18.3
- net G8: now also DD15.4
- net G9: now also DD15.12
- net GND: now also DD15.1, DD15.15, DD16.1, DD16.15, DD17.1, DD17.15, DD18.1, DD18.12, DD18.15
- net N$29: now also DD2.11, DD2.4, RD1.1
- net N$31: now also DD18.13
- net VCC: no longer DD14.14, DD15.16, DD16.16, DD17.16, DD18.16, DD19.16, DD20.14

Commit message: ..
Parts:
- moved RD1 8.52 mm to (184.2, 132.1), flipped to the bottom, turned to 270 degrees
Routing:
- net N$29: track 0.00 -> 33.1 mm
- net +5V: track 0.00 -> 2.41 mm
Changed lines of the file:
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@@
 <element name="R10" library="rcl" package="M1206" value="2k" x="234.95" y="167.64" rot="MR0"/>
 <element name="C7" library="rcl" package="E2,5-5" value="100m" x="234.95" y="161.29"/>
-<element name="RD1" library="rcl" package="M1206" value="2k" x="180.34" y="124.46"/>
+<element name="RD1" library="rcl" package="M1206" value="2k" x="184.15" y="132.08" rot="MR270"/>
 <element name="RD2" library="rcl" package="M1206" value="2k" x="185.42" y="92.71"/>
 </elements>
@@
 <wire x1="157.48" y1="109.22" x2="157.48" y2="127" width="0" layer="19" extent="1-1"/>
 <wire x1="180.34" y1="110.49" x2="157.48" y2="109.22" width="0" layer="19" extent="1-1"/>
-<wire x1="181.74" y1="124.46" x2="180.34" y2="110.49" width="0" layer="19" extent="1-1"/>
-<wire x1="184.15" y1="128.27" x2="181.74" y2="124.46" width="0" layer="19" extent="1-1"/>
+<wire x1="184.15" y1="130.68" x2="180.34" y2="110.49" width="0" layer="19" extent="1-1"/>
 <wire x1="184.02" y1="92.71" x2="180.34" y2="110.49" width="0" layer="19" extent="1-1"/>
 <wire x1="181.61" y1="90.17" x2="184.02" y2="92.71" width="0" layer="19" extent="1-1"/>
@@
 <wire x1="193.04" y1="199.52" x2="173.99" y2="177.8" width="0" layer="19" extent="16-16"/>
 <wire x1="227.33" y1="54.61" x2="207.01" y2="83.82" width="0" layer="19" extent="1-1"/>
+<wire x1="184.15" y1="130.68" x2="184.15" y2="128.27" width="0.4064" layer="16"/>
 </signal>
 <signal name="+12V">
@@
 <contactref element="RD1" pad="1"/>
 <contactref element="DD2" pad="4"/>
-<wire x1="176.53" y1="135.89" x2="184.15" y2="135.89" width="0" layer="19" extent="1-1"/>
-<wire x1="181.61" y1="128.27" x2="184.15" y2="135.89" width="0" layer="19" extent="1-1"/>
-<wire x1="178.94" y1="124.46" x2="181.61" y2="128.27" width="0" layer="19" extent="1-1"/>
-<wire x1="171.45" y1="128.27" x2="178.94" y2="124.46" width="0" layer="19" extent="1-1"/>
-<wire x1="168.91" y1="128.27" x2="171.45" y2="128.27" width="0" layer="19" extent="1-1"/>
-<wire x1="166.37" y1="128.27" x2="168.91" y2="128.27" width="0" layer="19" extent="1-1"/>
+<wire x1="181.61" y1="133.35" x2="181.61" y2="130.81" width="0.4064" layer="16"/>
+<wire x1="181.61" y1="130.81" x2="181.61" y2="128.27" width="0.4064" layer="16"/>
+<wire x1="166.37" y1="128.27" x2="166.37" y2="130.81" width="0.4064" layer="16"/>
+<wire x1="166.37" y1="130.81" x2="168.91" y2="130.81" width="0.4064" layer="16"/>
+<wire x1="168.91" y1="130.81" x2="168.91" y2="128.27" width="0.4064" layer="16"/>
+<wire x1="171.45" y1="128.27" x2="171.45" y2="130.81" width="0.4064" layer="16"/>
+<wire x1="171.45" y1="130.81" x2="168.91" y2="130.81" width="0.4064" layer="16"/>
+<wire x1="171.45" y1="130.81" x2="181.61" y2="130.81" width="0.4064" layer="16"/>
+<wire x1="184.15" y1="133.35" x2="184.15" y2="133.48" width="0.4064" layer="16"/>
+<wire x1="184.15" y1="133.48" x2="184.15" y2="135.89" width="0.4064" layer="16"/>
+<wire x1="181.61" y1="133.35" x2="184.02" y2="133.35" width="0.4064" layer="16"/>
+<wire x1="184.02" y1="133.35" x2="184.15" y2="133.48" width="0.4064" layer="16"/>
+<wire x1="181.61" y1="133.35" x2="176.53" y2="135.89" width="0" layer="19" extent="16-16"/>
 </signal>
 <signal name="N$33">
