File: SpecialistEE20.brd (EAGLE design)
At the start: 102 parts, among them IC1 74393N

Commit message: .
Parts:
- removed IC1: 74393N, 74xx-eu:DIL14
- added DD45: К555ИЕ19, 74xx-eu:DIL14
Connections:
- new net N$30: DD45.3
- new net N$47: DD45.4
- new net N$61: DD45.5
- new net N$62: DD45.11
- new net N$63: DD45.10
- new net N$64: DD45.1
- new net N$65: DD45.12, DD45.2
- net D0: now also DD112.34
- net D1: now also DD112.33
- net D2: now also DD112.32
- net D3: now also DD112.31
- net D4: now also DD112.30
- net D5: now also DD112.29
- net D6: now also DD112.28
- net D7: now also DD112.27
- net GND: now also DD45.7; no longer IC1.7
- net N$32: now also DD45.13, DD45.6; no longer IC1.13, IC1.6
- net VCC: now also DD45.14; no longer IC1.14
Changed lines of the file:
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@@
 <element name="DD3011.2" library="Разъёмы штырьковые 2.54мм" package="1X20" value="" x="86.36" y="167.64" rot="R270"/>
 <element name="KB" library="Speccy" package="MINI-DIN6" value="MINI-DIN6" x="57.15" y="213.36"/>
-<element name="IC1" library="74xx-eu" package="DIL14" value="74393N" x="229.87" y="130.81" rot="R90"/>
+<element name="DD45" library="74xx-eu" package="DIL14" value="К555ИЕ19" x="179.07" y="207.01" rot="R90"/>
 <element name="R105" library="rcl" package="M0805" value="4k7" x="54.61" y="210.82" rot="MR0"/>
 <element name="R106" library="rcl" package="M0805" value="4k7" x="64.77" y="212.09" rot="MR0"/>
@@
 <contactref element="DD103" pad="16"/>
 <contactref element="DD104" pad="16"/>
-<contactref element="IC1" pad="7"/>
+<contactref element="DD45" pad="7"/>
 <contactref element="DD113" pad="21"/>
 <contactref element="DD113" pad="3"/>
@@
 <wire x1="232.73" y1="186.69" x2="232.73" y2="173.99" width="0" layer="19" extent="16-16"/>
 <wire x1="236.22" y1="161.29" x2="232.73" y2="173.99" width="0" layer="19" extent="16-16"/>
-<wire x1="233.68" y1="138.43" x2="236.22" y2="161.29" width="0" layer="19" extent="1-1"/>
+<wire x1="182.88" y1="214.63" x2="236.22" y2="161.29" width="0" layer="19" extent="1-1"/>
 <wire x1="60.55" y1="204.86" x2="48.7426" y2="180.27" width="0" layer="19" extent="16-16"/>
 <wire x1="82.55" y1="213.36" x2="60.55" y2="204.86" width="0" layer="19" extent="1-1"/>
@@
 <contactref element="DD112" pad="26"/>
 <contactref element="DD31-" pad="24"/>
-<contactref element="IC1" pad="14"/>
+<contactref element="DD45" pad="14"/>
 <contactref element="27512" pad="28"/>
 <wire x1="95.25" y1="165.1" x2="82.55" y2="156.21" width="0" layer="19" extent="1-1"/>
@@
 <wire x1="77.47" y1="44.45" x2="62.23" y2="121.92" width="0" layer="19" extent="1-1"/>
 <wire x1="208.28" y1="116.84" x2="109.22" y2="127" width="0" layer="19" extent="1-1"/>
-<wire x1="226.06" y1="123.19" x2="208.28" y2="116.84" width="0" layer="19" extent="1-1"/>
+<wire x1="175.26" y1="199.39" x2="208.28" y2="116.84" width="0" layer="19" extent="1-1"/>
 </signal>
 <signal name="VSS/GND">
@@
 </signal>
 <signal name="N$32">
-<contactref element="IC1" pad="6"/>
-<contactref element="IC1" pad="13"/>
-<wire x1="226.06" y1="125.73" x2="233.68" y2="135.89" width="0" layer="19" extent="1-1"/>
+<contactref element="DD45" pad="6"/>
+<contactref element="DD45" pad="13"/>
+<wire x1="175.26" y1="201.93" x2="182.88" y2="212.09" width="0" layer="19" extent="1-1"/>
 </signal>
 <signal name="N$35">
@@
 <signal name="D0">
 <contactref element="DD3011.2" pad="7"/>
+<contactref element="DD112" pad="34"/>
+<wire x1="86.36" y1="176.53" x2="50.8" y2="184.15" width="0" layer="19" extent="1-1"/>
 </signal>
 <signal name="D1">
 <contactref element="DD3011.2" pad="8"/>
+<contactref element="DD112" pad="33"/>
+<wire x1="86.36" y1="173.99" x2="50.8" y2="181.61" width="0" layer="19" extent="1-1"/>
 </signal>
 <signal name="D2">
 <contactref element="DD3011.2" pad="9"/>
+<contactref element="DD112" pad="32"/>
+<wire x1="86.36" y1="171.45" x2="50.8" y2="179.07" width="0" layer="19" extent="1-1"/>
 </signal>
 <signal name="D3">
 <contactref element="DD3011.2" pad="10"/>
+<contactref element="DD112" pad="31"/>
+<wire x1="86.36" y1="168.91" x2="50.8" y2="176.53" width="0" layer="19" extent="1-1"/>
 </signal>
 <signal name="D4">
 <contactref element="DD3011.2" pad="11"/>
+<contactref element="DD112" pad="30"/>
+<wire x1="50.8" y1="173.99" x2="86.36" y2="166.37" width="0" layer="19" extent="1-1"/>
 </signal>
 <signal name="D5">
 <contactref element="DD3011.2" pad="12"/>
+<contactref element="DD112" pad="29"/>
+<wire x1="50.8" y1="171.45" x2="86.36" y2="163.83" width="0" layer="19" extent="1-1"/>
 </signal>
 <signal name="D6">
 <contactref element="DD3011.2" pad="13"/>
+<contactref element="DD112" pad="28"/>
+<wire x1="50.8" y1="168.91" x2="86.36" y2="161.29" width="0" layer="19" extent="1-1"/>
 </signal>
 <signal name="D7">
 <contactref element="DD3011.2" pad="14"/>
+<contactref element="DD112" pad="27"/>
+<wire x1="50.8" y1="166.37" x2="86.36" y2="158.75" width="0" layer="19" extent="1-1"/>
 </signal>
 <signal name="K27">
@@
 <contactref element="DD112" pad="6"/>
 </signal>
+<signal name="N$30">
+<contactref element="DD45" pad="3"/>
+</signal>
+<signal name="N$47">
+<contactref element="DD45" pad="4"/>
+</signal>
+<signal name="N$61">
+<contactref element="DD45" pad="5"/>
+</signal>
+<signal name="N$62">
+<contactref element="DD45" pad="11"/>
+</signal>
+<signal name="N$63">
+<contactref element="DD45" pad="10"/>
+</signal>
+<signal name="N$64">
+<contactref element="DD45" pad="1"/>
+</signal>
+<signal name="N$65">
+<contactref element="DD45" pad="2"/>
+<contactref element="DD45" pad="12"/>
+<wire x1="175.26" y1="204.47" x2="182.88" y2="201.93" width="0" layer="19" extent="1-1"/>
+</signal>
 </signals>

Commit message: d
Parts:
- removed DD31-: К589ИР12, 589:DIL24-6
- moved DD107 135.9 mm to (94.0, 114.3)
- moved DD31 135.9 mm to (77.5, 118.1)
- moved DD318.1 135.9 mm to (69.8, 118.1)
- moved DD318.2 135.9 mm to (85.1, 118.1)
- moved U$1 69.5 mm to (430.5, 39.4)
- moved KB 16.9 mm to (73.7, 209.6)
- moved DD113 15.2 mm to (76.2, 170.2)
- moved R105 9.25 mm to (63.5, 213.4)
- moved 27512 5.68 mm to (96.5, 41.9)
- moved DD112 4.02 mm to (47.0, 174.0)
- moved DD30 4.02 mm to (71.1, 166.4)
Connections:
- net GND: no longer DD31-.12
- net VCC: no longer DD31-.24

Commit message: ..
Parts:
- added R14: 2k, rcl:M1206
- moved DD113 4.02 mm to (72.4, 168.9)
Connections:
- removed net CPU_F1: DD20.10, R48.1
- removed net CPU_F2: DD20.13, R47.1
- removed net VBB/-5V: DD29.11
- removed net VCC/+5V: DD29.20
- removed net VDD/+12V: DD29.28
- removed net VSS/GND: DD29.2
- new net F1: DD20.10, DD29.22, R48.1
- new net F2: DD20.13, DD29.15, R47.1
- new net N$66: DD29.23, R14.1
- new net RESET80: DD12.6, DD29.12
- net !RD: now also DD112.5
- net +12V: now also DD29.28
- net +5V: now also DD29.20, R14.2
- net -5V: now also DD29.11
- net D0: now also DD29.10
- net D1: now also DD29.9
- net D2: now also DD29.8
- net D3: now also DD29.7
- net D4: now also DD29.3
- net D5: now also DD29.4
- net D6: now also DD29.5
- net D7: now also DD29.6
- net GND: now also DD29.14, DD29.2
- net RES: now also DD112.35

Commit message: 8.
Parts:
- moved DD3011.2 7.73 mm to (85.1, 160.0)
- moved DD29 5.24 mm to (125.7, 133.3)
Connections:
- net RESET80 renamed RES80
- new net A11: DD29.40
- new net A12: DD29.37
- new net A13: DD29.38
- new net A14: DD29.39
- new net A15: DD29.36
- net !WR: now also DD29.18
- net A0: now also DD29.25
- net A1: now also DD29.26
- net A10: now also DD29.1
- net A2: now also DD29.27
- net A3: now also DD29.29
- net A4: now also DD29.30
- net A5: now also DD29.31
- net A6: now also DD29.32
- net A7: now also DD29.33
- net A8: now also DD29.34
- net A9: now also DD29.35
- net GND: now also DD29.13

Commit message: a
Parts:
- removed DD318.1, DD318.2: (no value), Разъёмы штырьковые 2.54мм:1X12
- moved DD36 22.2 mm to (148.6, 203.2)
- moved 27512 17.8 mm to (114.3, 41.9)
- moved DD19 9.25 mm to (149.9, 190.5)
- moved DD336.2 8.98 mm to (66.0, 123.2)
- moved DD336.1 7.18 mm to (49.5, 120.7)
- moved DD38 3.81 mm to (102.9, 182.9)
- moved DD107 2.54 mm to (91.4, 114.3)
Connections:
- removed net R1: DD318.1.2, DD318.2.11
- net !RAS: no longer DD318.1.1
- net +5V: now also DD32.14, DD33.14, DD34.20, DD36.16, DD40.16; no longer DD318.2.1
- net G19: no longer DD318.2.12
- net GND: no longer DD318.1.11, DD318.1.12
- net MD0: no longer DD318.1.3
- net MD1: no longer DD318.1.5
- net MD2: no longer DD318.1.7
- net MD3: no longer DD318.1.9
- net MD4: no longer DD318.2.9
- net MD5: no longer DD318.2.7
- net MD6: no longer DD318.2.5
- net MD7: no longer DD318.2.3
- net VCC: no longer DD32.14, DD33.14, DD34.20, DD36.16, DD40.16
- net VD0: no longer DD318.1.4
- net VD1: no longer DD318.1.6
- net VD2: no longer DD318.1.8
- net VD3: no longer DD318.1.10
- net VD4: no longer DD318.2.10
- net VD5: no longer DD318.2.8
- net VD6: no longer DD318.2.6
- net VD7: no longer DD318.2.4
Routing:
- net GND: track 161.3 -> 154.9 mm
- net +5V: track 162.2 -> 157.6 mm
- net VD7: track 4.58 -> 0.00 mm
- net VD5: track 4.58 -> 0.00 mm
- net VD2: track 4.58 -> 0.00 mm
- net VD0: track 4.58 -> 0.00 mm
- net MD7: track 12.6 -> 8.03 mm
- net MD5: track 12.6 -> 8.03 mm
- net MD2: track 12.6 -> 8.03 mm
- net MD0: track 12.6 -> 8.03 mm
- net VD6: track 3.81 -> 0.00 mm
- net VD4: track 3.81 -> 0.00 mm
- net VD3: track 3.81 -> 0.00 mm
- net VD1: track 3.81 -> 0.00 mm
- net MD6: track 11.8 -> 8.03 mm
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
Commit message: o
Parts:
- added DD19': К555АП4, 74xx-eu:DIL20
- added RD3: 2k, rcl:M1206
- moved DD19 38.4 mm to (154.9, 228.6)
Connections:
- new net N$67: DD19'.19, RD3.2
- new net RD: DD29.17
- net GND: now also DD19'.1, DD19'.10
- net VCC: now also DD19'.20
Changed lines of the file:
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@@
 <element name="DD39" library="memory" package="DIL28" value="К573РФ4" x="127" y="177.8" rot="R270"/>
 <element name="DD34" library="74xx-eu" package="DIL20" value="К555АП6" x="105.41" y="115.57" rot="R270"/>
-<element name="DD19" library="74xx-eu" package="DIL16" value="К155ЛП10" x="149.86" y="190.5" rot="R180"/>
+<element name="DD19" library="74xx-eu" package="DIL16" value="К155ЛП10" x="154.94" y="228.6" rot="R180"/>
 <element name="C1" library="rcl" package="C0805" value="300" x="200.66" y="81.28" rot="MR0"/>
 <element name="R1" library="rcl" package="M1206" value="390" x="204.47" y="78.74" rot="MR0"/>
@@
 <element name="R23" library="rcl" package="M1206" value="2k" x="-10.16" y="96.52" rot="R180"/>
 <element name="R14" library="rcl" package="M1206" value="2k" x="127" y="107.95" rot="MR0"/>
+<element name="DD19'" library="74xx-eu" package="DIL20" value="К555АП4" x="158.75" y="191.77"/>
+<element name="RD3" library="rcl" package="M1206" value="2k" x="-10.16" y="16.51"/>
 </elements>
 <signals>
@@
 <contactref element="DD36" pad="8"/>
 <contactref element="DD40" pad="8"/>
+<contactref element="DD19'" pad="10"/>
+<contactref element="DD19'" pad="1"/>
 <wire x1="69.07183125" y1="166.157515625" x2="75.708171875" y2="171.66248125" width="0" layer="19" extent="16-16"/>
 <wire x1="70.203203125" y1="165.02614375" x2="69.07183125" y2="166.157515625" width="0" layer="19" extent="16-16"/>
@@
 <wire x1="191.77" y1="179.07" x2="191.77" y2="163.83" width="0" layer="19" extent="1-1"/>
 <wire x1="142.24" y1="184.15" x2="139.7" y2="168.91" width="0" layer="19" extent="1-1"/>
-<wire x1="140.97" y1="194.31" x2="142.24" y2="184.15" width="0" layer="19" extent="1-1"/>
-<wire x1="139.7" y1="207.01" x2="140.97" y2="194.31" width="0" layer="19" extent="1-1"/>
-<wire x1="110.49" y1="196.85" x2="139.7" y2="207.01" width="0" layer="19" extent="1-1"/>
+<wire x1="146.05" y1="232.41" x2="142.24" y2="184.15" width="0" layer="19" extent="1-1"/>
+<wire x1="139.7" y1="207.01" x2="146.05" y2="232.41" width="0" layer="19" extent="1-1"/>
 <wire x1="139.7" y1="134.62" x2="139.7" y2="151.13" width="0" layer="19" extent="1-1"/>
 <wire x1="139.7" y1="116.84" x2="154.94" y2="109.22" width="0" layer="19" extent="1-1"/>
@@
 <wire x1="77.06" y1="201.05" x2="63.5" y2="176.53" width="0" layer="19" extent="1-1"/>
 <wire x1="82.55" y1="213.36" x2="77.06" y2="201.05" width="0" layer="19" extent="1-1"/>
+<wire x1="110.49" y1="196.85" x2="146.05" y2="232.41" width="0" layer="19" extent="1-1"/>
 <wire x1="12.7" y1="200.66" x2="39.37" y2="182.88" width="0" layer="19" extent="1-1"/>
 <wire x1="182.88" y1="214.63" x2="191.77" y2="179.07" width="0" layer="19" extent="1-1"/>
@@
 <wire x1="137.16" y1="51.94" x2="142.24" y2="51.94" width="0" layer="19" extent="1-1"/>
 <wire x1="130.81" y1="34.29" x2="137.16" y2="51.94" width="0" layer="19" extent="1-1"/>
+<wire x1="170.18" y1="187.96" x2="35.56" y2="96.52" width="0" layer="19" extent="1-1"/>
+<wire x1="147.32" y1="187.96" x2="170.18" y2="187.96" width="0" layer="19" extent="1-1"/>
 </signal>
 <signal name="VCC">
@@
 <contactref element="DD45" pad="14"/>
 <contactref element="27512" pad="28"/>
+<contactref element="DD19'" pad="20"/>
 <wire x1="95.25" y1="168.91" x2="78.74" y2="154.94" width="0" layer="19" extent="1-1"/>
 <wire x1="54.61" y1="162.56" x2="78.74" y2="154.94" width="0" layer="19" extent="1-1"/>
@@
 <wire x1="175.26" y1="199.39" x2="134.62" y2="194.31" width="0" layer="19" extent="1-1"/>
 <wire x1="97.79" y1="49.53" x2="93.98" y2="132.08" width="0" layer="19" extent="1-1"/>
+<wire x1="147.32" y1="195.58" x2="97.79" y2="49.53" width="0" layer="19" extent="1-1"/>
 </signal>
 <signal name="N$3">
@@
 <wire x1="173.99" y1="177.8" x2="173.99" y2="166.37" width="0" layer="19" extent="1-1"/>
 <wire x1="157.48" y1="176.53" x2="173.99" y2="177.8" width="0" layer="19" extent="1-1"/>
-<wire x1="158.75" y1="186.69" x2="157.48" y2="176.53" width="0" layer="19" extent="1-1"/>
-<wire x1="157.48" y1="199.39" x2="158.75" y2="186.69" width="0" layer="19" extent="1-1"/>
+<wire x1="163.83" y1="224.79" x2="157.48" y2="176.53" width="0" layer="19" extent="1-1"/>
+<wire x1="157.48" y1="199.39" x2="163.83" y2="224.79" width="0" layer="19" extent="1-1"/>
 <wire x1="129.54" y1="203.07" x2="157.48" y2="199.39" width="0" layer="19" extent="16-16"/>
 <wire x1="157.48" y1="161.29" x2="157.48" y2="176.53" width="0" layer="19" extent="1-1"/>
@@
 <contactref element="DD29" pad="36"/>
 </signal>
+<signal name="RD">
+<contactref element="DD29" pad="17"/>
+</signal>
+<signal name="N$67">
+<contactref element="RD3" pad="2"/>
+<contactref element="DD19'" pad="19"/>
+<wire x1="-8.76" y1="16.51" x2="149.86" y2="195.58" width="0" layer="19" extent="1-1"/>
+</signal>
 </signals>

Commit message: d
Parts:
- moved 27512 125.8 mm to (109.2, 167.6)
- moved DD37 102.9 mm to (105.4, 248.9)
- moved DD38 100.5 mm to (108.0, 283.2)
- moved DD39 71.1 mm to (128.3, 248.9)
- moved DD19' 44.5 mm to (156.2, 236.2)
- moved DD107 30.5 mm to (100.3, 143.5)
- moved DD36 28.8 mm to (127.0, 184.2)
- moved KB 27.2 mm to (95.2, 193.0)
- moved DD32 24.4 mm to (61.0, 132.1)
- moved Z1 12.5 mm to (175.3, 85.1)
- moved DD19 11.5 mm to (153.7, 240.0)
- moved DD336.2 11.5 mm to (67.3, 111.8)
- moved DD3011.2 8.98 mm to (83.8, 168.9)
- moved DD112 8.89 mm to (47.0, 165.1)
- moved DD336.1 8.13 mm to (54.6, 114.3)
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Routing:
- net VID: track 405.2 -> 408.2 mm

Commit message: ..
Parts:
- moved RD3 285.3 mm to (146.1, 255.3)
- moved DD29 2.84 mm to (119.4, 129.5)
