File: SpecialistEE20.brd (EAGLE design)
At the start: 102 parts

Commit message: .
Parts:
- added DD13: К555ИР22, 74xx-eu:DIL20
- moved DD336.1 71.2 mm to (-16.5, 118.1)
- moved DD336.2 70.0 mm to (-2.54, 115.6)
- moved R8 28.1 mm to (31.8, 141.0), turned to 90 degrees
- moved DD107 27.7 mm to (92.7, 116.8)
- moved DD34 27.7 mm to (92.7, 143.5)
- moved DD113 19.4 mm to (68.6, 149.9), flipped to the top, turned to 270 degrees
- moved DD18 14.0 mm to (148.6, 151.1)
- moved R7 13.0 mm to (31.8, 146.1), turned to 90 degrees
- moved DD114 12.8 mm to (31.8, 180.3)
- moved DD12 12.7 mm to (142.2, 170.2)
- moved DD36 8.98 mm to (118.1, 185.4)
- moved DD17 8.89 mm to (148.6, 138.4)
- moved DD29 8.03 mm to (111.8, 132.1)
- moved DD3011.2 7.73 mm to (76.2, 167.6)
- moved 27512 6.48 mm to (102.9, 168.9)
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Connections:
- new net N$69: DD14.3, DD34.19
- new net N$70: DD12.9, DD14.2
- new net N$71: DD14.1
- net !RD: now also DD14.11, DD34.1
- net D0: now also DD34.2
- net D1: now also DD34.3
- net D2: now also DD34.9
- net D3: now also DD34.4
- net D4: now also DD34.5
- net D5: now also DD34.6
- net D6: now also DD34.7
- net D7: now also DD34.8
- net GND: now also DD13.10
- net MD0: now also DD34.18
- net MD1: now also DD34.17
- net MD2: now also DD34.11
- net MD3: now also DD34.16
- net MD4: now also DD34.15
- net MD5: now also DD34.14
- net MD6: now also DD34.13
- net MD7: now also DD34.12
- net RD: now also DD14.12, DD14.13
- net VCC: now also DD13.20
Routing:
- net GND: track 154.9 -> 392.8 mm
- net MA7: track 132.0 -> 205.8 mm
- net +5V: track 157.6 -> 228.3 mm
- net MA6: track 132.1 -> 202.0 mm
- net MA4: track 132.1 -> 191.3 mm
- net MA5: track 132.1 -> 187.3 mm
- net MA2: track 132.1 -> 179.4 mm
- net N$50: track 0.00 -> 42.3 mm
- net G19: track 0.00 -> 41.3 mm
- net MA3: track 132.1 -> 169.0 mm
- net N$56: track 0.00 -> 36.9 mm
- net MA0: track 132.1 -> 166.4 mm
- net VID: track 408.2 -> 375.0 mm
- net MA1: track 132.1 -> 162.5 mm
- net N$51: track 0.00 -> 30.0 mm
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
Commit message: 1
Parts:
- moved DD19 363.5 mm to (297.2, -94.0)
- moved DD19' 363.5 mm to (299.7, -97.8)
- moved DD37 363.5 mm to (248.9, -85.1)
- moved DD38 363.5 mm to (251.5, -50.8)
- moved DD39 363.5 mm to (271.8, -85.1)
- moved DD45 363.5 mm to (322.6, -127.0)
- moved R105 363.5 mm to (207.0, -120.7)
- moved R106 363.5 mm to (208.3, -121.9)
- moved R13 363.5 mm to (273.1, -129.5)
- moved RD3 363.5 mm to (289.6, -78.7)
- moved VD4 363.5 mm to (252.7, -129.5)
- moved VD5 363.5 mm to (257.8, -129.5)
- moved VD6 363.5 mm to (262.9, -129.5)
- moved VD7 363.5 mm to (268.0, -129.5)
- moved DD13 146.2 mm to (90.2, 11.4)
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Routing:
- net VID: track 375.0 -> 355.6 mm

Commit message: .
Parts:
- moved DD45 293.0 mm to (257.8, 158.8)
Changed lines of the file:
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@@
 <element name="DD3011.2" library="Разъёмы штырьковые 2.54мм" package="1X20" value="" x="76.2" y="167.64" rot="R270"/>
 <element name="KB" library="Speccy" package="MINI-DIN6" value="MINI-DIN6" x="95.25" y="193.04"/>
-<element name="DD45" library="74xx-eu" package="DIL14" value="К555ИЕ19" x="322.58" y="-127" rot="R90"/>
+<element name="DD45" library="74xx-eu" package="DIL14" value="К555ИЕ19" x="257.81" y="158.75" rot="R90"/>
 <element name="R105" library="rcl" package="M0805" value="4k7" x="207.01" y="-120.65" rot="MR0"/>
 <element name="R106" library="rcl" package="M0805" value="4k7" x="208.28" y="-121.92" rot="MR0"/>
@@
 <wire x1="288.29" y1="-90.17" x2="288.29" y2="-101.6" width="0" layer="19" extent="1-1"/>
 <wire x1="311.15" y1="-101.6" x2="288.29" y2="-101.6" width="0" layer="19" extent="1-1"/>
-<wire x1="326.39" y1="-119.38" x2="311.15" y2="-101.6" width="0" layer="19" extent="1-1"/>
+<wire x1="261.62" y1="166.37" x2="311.15" y2="-101.6" width="0" layer="19" extent="1-1"/>
 </signal>
 <signal name="VCC">
@@
 <wire x1="243.84" y1="-64.77" x2="279.4" y2="-68.58" width="0" layer="19" extent="1-1"/>
 <wire x1="241.3" y1="-99.06" x2="243.84" y2="-64.77" width="0" layer="19" extent="1-1"/>
-<wire x1="318.77" y1="-134.62" x2="288.29" y2="-93.98" width="0" layer="19" extent="1-1"/>
+<wire x1="254" y1="151.13" x2="288.29" y2="-93.98" width="0" layer="19" extent="1-1"/>
 <wire x1="93.98" y1="22.86" x2="243.84" y2="-64.77" width="0" layer="19" extent="1-1"/>
 <wire x1="76.2" y1="156.21" x2="93.98" y2="22.86" width="0" layer="19" extent="1-1"/>
@@
 <contactref element="DD45" pad="6"/>
 <contactref element="DD45" pad="13"/>
-<wire x1="318.77" y1="-132.08" x2="326.39" y2="-121.92" width="0" layer="19" extent="1-1"/>
+<wire x1="254" y1="153.67" x2="261.62" y2="163.83" width="0" layer="19" extent="1-1"/>
 </signal>
 <signal name="N$35">
@@
 <contactref element="DD45" pad="2"/>
 <contactref element="DD45" pad="12"/>
-<wire x1="318.77" y1="-129.54" x2="326.39" y2="-132.08" width="0" layer="19" extent="1-1"/>
+<wire x1="254" y1="156.21" x2="261.62" y2="153.67" width="0" layer="19" extent="1-1"/>
 </signal>
 <signal name="RES80">

Commit message: g
Connections:
- net N$44 renamed !G19B
- net N$70 renamed !G19A
- removed net N$36: DD12.12
- new net SNY: DD12.12, DD29.19
Changed lines of the file:
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@@
 <wire x1="147.32" y1="173.99" x2="233.68" y2="161.29" width="0" layer="19" extent="1-1"/>
-</signal>
-<signal name="N$36">
-<contactref element="DD12" pad="12"/>
 </signal>
 <signal name="N$37">
@@
 <wire x1="27.94" y1="102.87" x2="78.74" y2="109.22" width="0" layer="19" extent="1-1"/>
 </signal>
-<signal name="N$44">
+<signal name="!G19B">
 <contactref element="DD107" pad="4"/>
 <contactref element="DD107" pad="3"/>
@@
 <wire x1="148.59" y1="186.69" x2="96.52" y2="152.4" width="0" layer="19" extent="1-1"/>
 </signal>
-<signal name="N$70">
+<signal name="N$71">
+<contactref element="DD14" pad="1"/>
+</signal>
+<signal name="SNY">
+<contactref element="DD29" pad="19"/>
+<contactref element="DD12" pad="12"/>
+<wire x1="144.78" y1="166.37" x2="104.14" y2="110.49" width="0" layer="19" extent="1-1"/>
+</signal>
+<signal name="!G19A">
 <contactref element="DD12" pad="9"/>
 <contactref element="DD14" pad="2"/>
 <wire x1="137.16" y1="166.37" x2="151.13" y2="186.69" width="0" layer="19" extent="1-1"/>
 </signal>
-<signal name="N$71">
-<contactref element="DD14" pad="1"/>
-</signal>
 </signals>

Commit message: .
Parts:
- removed DD336.1, DD336.2: (no value), Разъёмы штырьковые 2.54мм:1X07
- added JP2: (no value), Разъёмы штырьковые 2.54мм:1X30
- added JP3, JP4: (no value), Разъёмы штырьковые 2.54мм:1X20
- added X1: SCART-F, con-hirschmann:SCART-F
- DD13: value К555ИР22 -> КР580ВВ55; device 74xx-eu:DIL20 -> micro-intel:DIL40
- moved 27512 187.5 mm to (-49.5, 59.7), turned to 270 degrees
- moved DD13 94.6 mm to (-2.54, 30.5)
- moved DD114 63.9 mm to (54.6, 120.7)
- moved DD32 50.0 mm to (106.7, 111.8)
- moved DD113 34.9 mm to (74.9, 115.6)
- moved DD112 34.9 mm to (54.6, 133.3)
- moved DD30 34.9 mm to (74.9, 133.3)
- moved DD3011.1 34.9 mm to (67.3, 133.3)
- moved DD3011.2 34.9 mm to (82.5, 133.3)
- moved DD33 30.6 mm to (91.4, 114.3)
- moved DD31 28.0 mm to (96.5, 138.4)
- moved DD107 19.8 mm to (77.5, 104.1), turned to 0 degrees
- moved DD34 17.7 mm to (109.2, 137.2)
- moved DD29 14.2 mm to (125.7, 129.5)
- moved KB 5.08 mm to (100.3, 193.0)
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Connections:
- removed net N$53: DD32.9, DD33.9, DD9.12
- removed net N$57: DD32.6, DD33.6, DD9.4
- removed net SH: DD336.1.1
- removed net VD10: DD336.1.4
- removed net VD11: DD336.1.5
- removed net VD8: DD336.1.2
- removed net VD9: DD336.1.3
- net +5V: no longer DD336.2.1
- net CLK: now also DD32.9, DD33.9, DD9.12; no longer DD336.2.6
- net GND: now also DD13.7; no longer DD13.10, DD336.1.7
- net Q3: now also DD32.6, DD33.6, DD9.4; no longer DD336.1.6
- net R2: no longer DD336.2.7
- net VCC: now also DD13.26; no longer DD13.20
- net VID: no longer DD336.2.5
Routing:
- net !RD: track 21.4 -> 27.5 mm
Other:
- board outline added: 55.9 x 6.6 mm

Commit message: 9
Parts:
- removed DD13: КР580ВВ55, micro-intel:DIL40
- removed DD19': К555АП4, 74xx-eu:DIL20
- removed JP2: (no value), Разъёмы штырьковые 2.54мм:1X30
- removed JP3, JP4: (no value), Разъёмы штырьковые 2.54мм:1X20
- removed RD3: 2k, rcl:M1206
- added J1: (no value), Speccy:SDCMF-10915W010
- added R103: (no value), rcl:RTRIM3296W
- added U$2: SWITCH9X4, ESR_NM8032:SWITCH9X4
- R9: value (none) -> 2k; device rcl:RTRIM3296W -> rcl:M1206
- moved R9 370.1 mm to (273.1, -129.5), flipped to the bottom, turned to 270 degrees
- moved R13 341.7 mm to (-68.6, -135.9), flipped to the top, turned to 0 degrees
- moved DD114 8.89 mm to (54.6, 129.5), flipped to the top, turned to 90 degrees
- renumbered R7 to R101, R8 to R102
Connections:
- removed net N$67: DD19'.19, RD3.2
- new net !R: DD114.24
- new net CS: DD114.14
- new net MISO: DD114.16
- new net MOSI: DD114.15
- new net N$36: DD20.3
- new net N$44: DD11.3, DD20.2
- new net N$53: DD20.1, DD9.5
- new net SCK: DD114.17
- new net TON: DD114.25
- new net VDD: J1.4
- new net VSS1: J1.3
- new net VSS2: J1.6
- net !RESIN: now also DD114.29
- net !WR: now also DD112.36
- net +5V: now also R9.2; no longer R13.2
- net A0: now also DD112.9
- net A1: now also DD112.8
- net GND: now also J1.M1, J1.M2, J1.M3, J1.M4, R103.3; no longer DD13.7, DD19'.1, DD19'.10, R9.3
- net N$18: now also R9.1; no longer R13.1
- net N$56: now also R103.1; no longer R9.1
- net N$60: now also R103.2; no longer R9.2
- net P17: now also DD114.30
- net P18: now also DD114.31
- net P19: now also DD114.32
- net P20: now also DD114.1
- net P21: now also DD114.2
- net P22: now also DD114.9
- net P23: now also DD114.10
- net P24: now also DD114.11
- net VCC: no longer DD13.26, DD19'.20

Commit message: .
Parts:
- moved R13 332.5 mm to (185.4, 78.7)
- moved R23 114.6 mm to (125.7, 115.6)
Connections:
- net N$36 renamed STRT
- removed net N$71: DD14.1
- new net DD9DD14: DD14.1, DD36.15, DD36.2, DD9.6
- net +5V: now also R13.2
- net A11: now also DD36.3
- net A12: now also DD36.13
- net A13: now also DD36.1, DD36.14
- net A14: now also DD11.1
- net A15: now also DD11.2
- net N$53: now also R13.1
Changed lines of the file:
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@@
 <element name="R107" library="rcl" package="M0805" value="560" x="11.43" y="191.77" rot="MR90"/>
 <element name="27512" library="memory" package="DIL28" value="" x="-49.53" y="59.69" rot="R270"/>
-<element name="R23" library="rcl" package="M1206" value="2k" x="58.42" y="22.86" rot="R180"/>
+<element name="R23" library="rcl" package="M1206" value="2k" x="125.73" y="115.57" rot="R180"/>
 <element name="R14" library="rcl" package="M1206" value="2k" x="127" y="107.95" rot="MR0"/>
 <element name="X1" library="con-hirschmann" package="SCART-F" value="SCART-F" x="58.42" y="181.61" rot="R180">
@@
 <element name="J1" library="Speccy" package="SDCMF-10915W010" value="" x="-2.54" y="172.72" rot="R180"/>
 <element name="U$2" library="ESR_NM8032" package="SWITCH9X4" value="SWITCH9X4" x="-12.7" y="152.4"/>
-<element name="R13" library="rcl" package="M1206" value="2k" x="-68.58" y="-135.89"/>
+<element name="R13" library="rcl" package="M1206" value="2k" x="185.42" y="78.74"/>
 </elements>
 <signals>
@@
 <wire x1="85.09" y1="100.33" x2="86.36" y2="99.06" width="0" layer="19" extent="16-16"/>
 <wire x1="87.63" y1="106.68" x2="85.09" y2="100.33" width="0" layer="19" extent="1-1"/>
-<wire x1="10.906125" y1="161.29" x2="25.4" y2="151.13" width="0" layer="19" extent="1-16"/>
 <wire x1="167.64" y1="105.41" x2="162.56" y2="99.06" width="0" layer="19" extent="16-16"/>
 <wire x1="137.16" y1="107.95" x2="137.16" y2="99.06" width="0" layer="19" extent="16-16"/>
@@
 <wire x1="74.53" y1="119.8626" x2="76.13" y2="119.8626" width="0" layer="19" extent="1-1"/>
 <wire x1="193.04" y1="149.86" x2="180.34" y2="152.4" width="0" layer="19" extent="1-1"/>
-<wire x1="10.668" y1="175.26" x2="25.4" y2="151.13" width="0" layer="19" extent="1-16"/>
 <wire x1="191.77" y1="163.83" x2="193.04" y2="149.86" width="0" layer="19" extent="1-1"/>
 <wire x1="190.5" y1="135.89" x2="193.04" y2="149.86" width="0" layer="19" extent="1-1"/>
@@
 <wire x1="134.62" y1="173.99" x2="137.16" y2="157.48" width="0" layer="19" extent="16-16"/>
 <wire x1="138.43" y1="186.69" x2="134.62" y2="173.99" width="0" layer="19" extent="1-1"/>
+<wire x1="10.906125" y1="161.29" x2="25.4" y2="151.13" width="0" layer="19" extent="1-16"/>
+<wire x1="10.668" y1="175.26" x2="10.906125" y2="161.29" width="0" layer="19" extent="1-1"/>
 <wire x1="193.04" y1="181.61" x2="191.77" y2="163.83" width="0" layer="19" extent="1-1"/>
 <wire x1="118.11" y1="151.13" x2="137.16" y2="154.94" width="0" layer="19" extent="16-16"/>
+<wire x1="12.7" y1="200.66" x2="10.668" y2="175.26" width="0" layer="19" extent="1-1"/>
 <wire x1="113.03" y1="189.23" x2="138.43" y2="186.69" width="0" layer="19" extent="1-1"/>
 <wire x1="103.73" y1="184.54" x2="113.03" y2="189.23" width="0" layer="19" extent="1-1"/>
@@
 <wire x1="236.22" y1="161.29" x2="232.73" y2="173.99" width="0" layer="19" extent="16-16"/>
 <wire x1="261.62" y1="166.37" x2="236.22" y2="161.29" width="0" layer="19" extent="1-1"/>
-<wire x1="12.7" y1="200.66" x2="10.668" y2="175.26" width="0" layer="19" extent="1-1"/>
 <wire x1="162.56" y1="55.04" x2="162.56" y2="96.52" width="0" layer="19" extent="1-1"/>
 <wire x1="152.4" y1="55.04" x2="162.56" y2="55.04" width="0" layer="19" extent="1-1"/>
@@
 <wire x1="45.72" y1="125.73" x2="45.72" y2="118.11" width="0.4064" layer="16"/>
 <wire x1="45.72" y1="118.11" x2="43.18" y2="115.57" width="0.4064" layer="16"/>
+<contactref element="R13" pad="2"/>
 <wire x1="113.03" y1="148.59" x2="100.33" y2="149.86" width="0" layer="19" extent="1-1"/>
 <wire x1="95.25" y1="121.92" x2="100.33" y2="149.86" width="0" layer="19" extent="1-1"/>
@@
 <wire x1="69.85" y1="107.95" x2="72.93" y2="111.2774" width="0" layer="19" extent="1-1"/>
 <wire x1="110.49" y1="119.38" x2="95.25" y2="121.92" width="0" layer="19" extent="1-1"/>
-<wire x1="118.11" y1="105.41" x2="110.49" y2="119.38" width="0" layer="19" extent="1-1"/>
-<wire x1="125.6" y1="107.95" x2="118.11" y2="105.41" width="0" layer="19" extent="16-16"/>
+<wire x1="124.33" y1="115.57" x2="110.49" y2="119.38" width="0" layer="19" extent="1-1"/>
+<wire x1="125.6" y1="107.95" x2="124.33" y2="115.57" width="0" layer="19" extent="1-16"/>
+<wire x1="118.11" y1="105.41" x2="125.6" y2="107.95" width="0" layer="19" extent="16-16"/>
 <wire x1="55.81" y1="125.2474" x2="73.73" y2="119.8626" width="0" layer="19" extent="1-1"/>
 <wire x1="54.21" y1="125.2474" x2="55.81" y2="125.2474" width="0" layer="19" extent="1-1"/>
@@
 <wire x1="182.88" y1="97.79" x2="180.34" y2="110.49" width="0" layer="19" extent="1-1"/>
 <wire x1="184.02" y1="92.71" x2="182.88" y2="97.79" width="0" layer="19" extent="1-1"/>
+<wire x1="186.82" y1="78.74" x2="184.02" y2="92.71" width="0" layer="19" extent="1-1"/>
 <wire x1="184.15" y1="128.27" x2="180.34" y2="110.49" width="0" layer="19" extent="1-1"/>
-<wire x1="205.74" y1="128.27" x2="184.15" y2="128.27" width="0" layer="19" extent="1-1"/>
+<wire x1="205.74" y1="83.82" x2="186.82" y2="78.74" width="0" layer="19" extent="1-1"/>
+<wire x1="207.01" y1="97.79" x2="205.74" y2="83.82" width="0" layer="19" extent="1-1"/>
+<wire x1="205.74" y1="110.49" x2="207.01" y2="97.79" width="0" layer="19" extent="1-1"/>
+<wire x1="205.74" y1="128.27" x2="205.74" y2="110.49" width="0" layer="19" extent="1-1"/>
 <wire x1="208.28" y1="142.24" x2="205.74" y2="128.27" width="0" layer="19" extent="1-1"/>
 <wire x1="207.01" y1="156.21" x2="208.28" y2="142.24" width="0" layer="19" extent="1-1"/>
-<wire x1="205.74" y1="110.49" x2="205.74" y2="128.27" width="0" layer="19" extent="1-1"/>
-<wire x1="207.01" y1="97.79" x2="205.74" y2="110.49" width="0" layer="19" extent="1-1"/>
-<wire x1="205.74" y1="83.82" x2="207.01" y2="97.79" width="0" layer="19" extent="1-1"/>
 <wire x1="208.28" y1="173.99" x2="207.01" y2="156.21" width="0" layer="19" extent="1-1"/>
 <wire x1="220.98" y1="169.04" x2="208.28" y2="173.99" width="0" layer="19" extent="16-16"/>
@@
 <wire x1="96.93" y1="184.54" x2="130.81" y2="181.61" width="0" layer="19" extent="1-1"/>
 <wire x1="227.33" y1="54.61" x2="205.74" y2="83.82" width="0" layer="19" extent="1-1"/>
-<wire x1="57.02" y1="22.86" x2="52.07" y2="76.2" width="0" layer="19" extent="1-16"/>
 <wire x1="306.07" y1="-97.79" x2="227.33" y2="54.61" width="0" layer="19" extent="1-1"/>
 <wire x1="273.05" y1="-130.94" x2="306.07" y2="-97.79" width="0" layer="19" extent="16-16"/>
@@
 <contactref element="DD32" pad="8"/>
 <contactref element="R23" pad="1"/>
+<wire x1="110.49" y1="104.14" x2="127.13" y2="115.57" width="0" layer="19" extent="1-1"/>
 <wire x1="95.25" y1="106.68" x2="110.49" y2="104.14" width="0" layer="19" extent="1-1"/>
-<wire x1="59.82" y1="22.86" x2="95.25" y2="106.68" width="0" layer="19" extent="1-1"/>
 </signal>
 <signal name="!U6">
@@
 <signal name="A11">
 <contactref element="DD29" pad="40"/>
+<contactref element="DD36" pad="3"/>
+<wire x1="133.35" y1="153.67" x2="125.73" y2="189.23" width="0" layer="19" extent="1-1"/>
 </signal>
 <signal name="A12">
 <contactref element="DD29" pad="37"/>
+<contactref element="DD36" pad="13"/>
+<wire x1="133.35" y1="146.05" x2="123.19" y2="181.61" width="0" layer="19" extent="1-1"/>
 </signal>
 <signal name="A13">
 <contactref element="DD29" pad="38"/>
+<contactref element="DD36" pad="14"/>
+<contactref element="DD36" pad="1"/>
+<wire x1="125.73" y1="181.61" x2="130.81" y2="189.23" width="0" layer="19" extent="1-1"/>
+<wire x1="133.35" y1="148.59" x2="125.73" y2="181.61" width="0" layer="19" extent="1-1"/>
 </signal>
 <signal name="A14">
 <contactref element="DD29" pad="39"/>
+<contactref element="DD11" pad="1"/>
+<wire x1="133.35" y1="151.13" x2="208.28" y2="181.61" width="0" layer="19" extent="1-1"/>
 </signal>
 <signal name="A15">
 <contactref element="DD29" pad="36"/>
+<contactref element="DD11" pad="2"/>
+<wire x1="133.35" y1="143.51" x2="205.74" y2="181.61" width="0" layer="19" extent="1-1"/>
 </signal>
 <signal name="RD">
@@
 <wire x1="113.03" y1="146.05" x2="148.59" y2="186.69" width="0" layer="19" extent="1-1"/>
 </signal>
-<signal name="N$71">
-<contactref element="DD14" pad="1"/>
-</signal>
 <signal name="SNY">
 <contactref element="DD29" pad="19"/>
@@
 <contactref element="DD114" pad="17"/>
 </signal>
-<signal name="N$36">
-<contactref element="DD20" pad="3"/>
-</signal>
 <signal name="N$44">
 <contactref element="DD20" pad="2"/>
@@
 <contactref element="DD20" pad="1"/>
 <contactref element="DD9" pad="5"/>
+<contactref element="R13" pad="1"/>
 <wire x1="172.72" y1="105.41" x2="180.34" y2="118.11" width="0" layer="19" extent="1-1"/>
+<wire x1="184.02" y1="78.74" x2="172.72" y2="105.41" width="0" layer="19" extent="1-1"/>
+</signal>
+<signal name="STRT">
+<contactref element="DD20" pad="3"/>
+</signal>
+<signal name="DD9DD14">
+<contactref element="DD36" pad="2"/>
+<contactref element="DD36" pad="15"/>
+<contactref element="DD9" pad="6"/>
+<contactref element="DD14" pad="1"/>
+<wire x1="128.27" y1="189.23" x2="153.67" y2="186.69" width="0" layer="19" extent="1-1"/>
+<wire x1="128.27" y1="181.61" x2="128.27" y2="189.23" width="0" layer="19" extent="1-1"/>
+<wire x1="170.18" y1="105.41" x2="153.67" y2="186.69" width="0" layer="19" extent="1-1"/>
 </signal>
 </signals>
