File: SpecialistEE20.brd (EAGLE design)
At the start: 55.9 x 6.6 mm, 102 parts, among them X1 SCART-F

Commit message: .
Parts:
- moved 27512 185.3 mm to (102.9, 165.1), turned to 0 degrees
Connections:
- net !G19A: now also DD7.3
- net !RD: now also DD7.5
- net !WE: now also DD7.6
- net G15: now also DD7.4
Changed lines of the file:
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@@
 <element name="LED1" library="led" package="LED5MM" value="" x="11.43" y="200.66"/>
 <element name="R107" library="rcl" package="M0805" value="560" x="11.43" y="191.77" rot="MR90"/>
-<element name="27512" library="memory" package="DIL28" value="" x="-49.53" y="59.69" rot="R270"/>
+<element name="27512" library="memory" package="DIL28" value="" x="102.87" y="165.1"/>
 <element name="R23" library="rcl" package="M1206" value="2k" x="125.73" y="115.57" rot="R180"/>
 <element name="R14" library="rcl" package="M1206" value="2k" x="127" y="107.95" rot="MR0"/>
@@
 <wire x1="10.906125" y1="161.29" x2="25.4" y2="151.13" width="0" layer="19" extent="1-16"/>
 <wire x1="10.668" y1="175.26" x2="10.906125" y2="161.29" width="0" layer="19" extent="1-1"/>
+<wire x1="119.38" y1="157.48" x2="137.16" y2="157.48" width="0" layer="19" extent="16-16"/>
+<wire x1="118.11" y1="151.13" x2="119.38" y2="157.48" width="0" layer="19" extent="1-1"/>
 <wire x1="193.04" y1="181.61" x2="191.77" y2="163.83" width="0" layer="19" extent="1-1"/>
-<wire x1="118.11" y1="151.13" x2="137.16" y2="154.94" width="0" layer="19" extent="16-16"/>
 <wire x1="12.7" y1="200.66" x2="10.668" y2="175.26" width="0" layer="19" extent="1-1"/>
 <wire x1="113.03" y1="189.23" x2="138.43" y2="186.69" width="0" layer="19" extent="1-1"/>
@@
 <wire x1="142.24" y1="51.94" x2="147.32" y2="55.04" width="0" layer="19" extent="1-1"/>
 <wire x1="137.16" y1="51.94" x2="142.24" y2="51.94" width="0" layer="19" extent="1-1"/>
-<wire x1="-57.15" y1="43.18" x2="33.02" y2="99.06" width="0" layer="19" extent="16-16"/>
 <wire x1="259.08" y1="-36.83" x2="162.56" y2="55.04" width="0" layer="19" extent="1-1"/>
 <wire x1="256.54" y1="-71.12" x2="259.08" y2="-36.83" width="0" layer="19" extent="1-1"/>
@@
 <wire x1="241.3" y1="-99.06" x2="243.84" y2="-64.77" width="0" layer="19" extent="1-1"/>
 <wire x1="254" y1="151.13" x2="243.84" y2="-64.77" width="0" layer="19" extent="1-1"/>
-<wire x1="82.55" y1="121.92" x2="254" y2="151.13" width="0" layer="19" extent="1-1"/>
-<wire x1="-41.91" y1="76.2" x2="62.23" y2="121.92" width="0" layer="19" extent="1-1"/>
+<wire x1="86.36" y1="172.72" x2="254" y2="151.13" width="0" layer="19" extent="1-1"/>
+<wire x1="78.74" y1="123.19" x2="86.36" y2="172.72" width="0" layer="19" extent="16-16"/>
 </signal>
 <signal name="N$3">
@@
 <contactref element="DD1" pad="1"/>
 <contactref element="C6" pad="1"/>
-<wire x1="200.66" y1="118.11" x2="234.63" y2="186.69" width="0" layer="19" extent="16-16"/>
+<contactref element="DD7" pad="4"/>
+<wire x1="199.39" y1="163.83" x2="234.63" y2="186.69" width="0" layer="19" extent="16-16"/>
+<wire x1="200.66" y1="118.11" x2="199.39" y2="163.83" width="0" layer="19" extent="1-1"/>
 <wire x1="204.47" y1="105.41" x2="200.66" y2="118.11" width="0" layer="19" extent="1-1"/>
 <wire x1="205.74" y1="91.44" x2="204.47" y2="105.41" width="0" layer="19" extent="1-1"/>
@@
 <wire x1="69.85" y1="91.44" x2="72.39" y2="90.17" width="0.4064" layer="16"/>
 <wire x1="72.39" y1="90.17" x2="74.93" y2="90.17" width="0.4064" layer="16"/>
+<contactref element="DD7" pad="6"/>
+<wire x1="194.31" y1="163.83" x2="154.94" y2="91.44" width="0" layer="19" extent="1-1"/>
 </signal>
 <signal name="MD1">
@@
 <wire x1="59.69" y1="139.7" x2="48.26" y2="148.59" width="0.4064" layer="16"/>
 <wire x1="48.26" y1="148.59" x2="46.99" y2="147.32" width="0.4064" layer="16"/>
+<contactref element="DD7" pad="5"/>
 <wire x1="67.31" y1="147.32" x2="105.41" y2="148.59" width="0" layer="19" extent="1-1"/>
 <wire x1="146.05" y1="179.07" x2="105.41" y2="148.59" width="0" layer="19" extent="1-1"/>
+<wire x1="196.85" y1="163.83" x2="146.05" y2="179.07" width="0" layer="19" extent="1-1"/>
 </signal>
 <signal name="N$40">
@@
 <contactref element="DD12" pad="9"/>
 <contactref element="DD14" pad="2"/>
+<contactref element="DD7" pad="3"/>
+<wire x1="151.13" y1="186.69" x2="201.93" y2="163.83" width="0" layer="19" extent="1-1"/>
 <wire x1="137.16" y1="166.37" x2="151.13" y2="186.69" width="0" layer="19" extent="1-1"/>
 </signal>
