File: SpecialistEE20.sch (EAGLE design)
At the start: 93 parts

Commit message: .
Parts:
- DD102, DD103, DD104, DD21, DD22, DD23, DD24, DD25, DD26, DD27, DD28: device ic-package:DIL16 -> memory:2164
- DD31: device ic-package:DIL24-6 -> 589:589IR12
Connections:
- new net !CAS: DD21.!CAS, DD22.!CAS, DD23.!CAS, DD24.!CAS, DD25.!CAS, DD26.!CAS, DD27.!CAS, DD28.!CAS
- new net !RAS: DD21.!RAS, DD22.!RAS, DD23.!RAS, DD24.!RAS, DD25.!RAS, DD26.!RAS, DD27.!RAS, DD28.!RAS
- new net !WE: DD21.!WE, DD22.!WE, DD23.!WE, DD24.!WE, DD25.!WE, DD26.!WE, DD27.!WE, DD28.!WE
- new net MD0: DD21.DI, DD21.DO
- new net MD1: DD22.DI, DD22.DO
- new net MD2: DD23.DI, DD23.DO
- new net MD3: DD24.DI, DD24.DO
- new net MD4: DD25.DI, DD25.DO
- new net MD5: DD26.DI, DD26.DO
- new net MD6: DD27.DI, DD27.DO
- new net MD7: DD28.DI, DD28.DO
- net +5V: now also DD102.VCC, DD103.VCC, DD104.VCC, DD21.VCC, DD22.VCC, DD23.VCC, DD24.VCC, DD25.VCC, DD26.VCC, DD27.VCC, DD28.VCC
- net GND: now also DD102.VSS, DD103.VSS, DD104.VSS, DD21.VSS, DD22.VSS, DD23.VSS, DD24.VSS, DD25.VSS, DD26.VSS, DD27.VSS, DD28.VSS
- net MA0: now also DD21.A0, DD22.A0, DD23.A0, DD24.A0, DD25.A0, DD26.A0, DD27.A0, DD28.A0
- net MA1: now also DD21.A1, DD22.A1, DD23.A1, DD24.A1, DD25.A1, DD26.A1, DD27.A1, DD28.A1
- net MA2: now also DD21.A2, DD22.A2, DD23.A2, DD24.A2, DD25.A2, DD26.A2, DD27.A2, DD28.A2
- net MA3: now also DD21.A3, DD22.A3, DD23.A3, DD24.A3, DD25.A3, DD26.A3, DD27.A3, DD28.A3
- net MA4: now also DD21.A4, DD22.A4, DD23.A4, DD24.A4, DD25.A4, DD26.A4, DD27.A4, DD28.A4
- net MA5: now also DD21.A5, DD22.A5, DD23.A5, DD24.A5, DD25.A5, DD26.A5, DD27.A5, DD28.A5
- net MA6: now also DD21.A6, DD22.A6, DD23.A6, DD24.A6, DD25.A6, DD26.A6, DD27.A6, DD28.A6
- net MA7: now also DD21.A7, DD22.A7, DD23.A7, DD24.A7, DD25.A7, DD26.A7, DD27.A7, DD28.A7
Other:
- moved on the sheet: DD32P

Commit message: k
Parts:
- removed DD111: КР580ВВ55, micro-intel:8255A
- added DD3011.1, DD3011.2: (no value), Разъёмы штырьковые 2.54мм:PINHD-1X20
- added IC1: 74393N, 74xx-eu:74393N
- added KB: MINI-DIN6, Speccy:MINI-DIN6PTH
- added R105, R106: 4k7, rcl:R-EU_M0805
Connections:
- new net !RD: DD3011.1.5
- new net !RESIN: DD113.PC6(/RESET)
- new net !U7: DD107C.I0, DD3011.1.6
- new net !WR: DD107C.I1, DD3011.2.5
- new net B: DD3011.1.13
- new net D0: DD3011.2.7
- new net D1: DD3011.2.8
- new net D2: DD3011.2.9
- new net D3: DD3011.2.10
- new net D4: DD3011.2.11
- new net D5: DD3011.2.12
- new net D6: DD3011.2.13
- new net D7: DD3011.2.14
- new net G: DD3011.1.11
- new net K1: DD113.PB3(MOSI/OC2), DD3011.1.1
- new net K10: DD113.PC4(ADC4/SDA), DD3011.2.17
- new net K11: DD113.PC3(ADC3), DD3011.2.18
- new net K12: DD113.PC2(ADC2), DD3011.2.19
- new net K13: DD113.PD0(RXD), DD3011.1.14
- new net K14: DD113.PD1(TXD), DD3011.1.15
- new net K15: DD113.PD4(XCK/T0), DD3011.1.16
- new net K16: DD113.PD5(T1), DD3011.1.17
- new net K17: DD113.PC1(ADC1), DD3011.2.20
- new net K18: DD113.PC0(ADC0), DD3011.1.20
- new net K19: DD113.PD7(AIN1), DD3011.1.19
- new net K2: DD113.PB2(SS/OC1B), DD3011.1.2
- new net K27: DD3011.1.18
- new net K3: DD113.PB1(OC1A), DD3011.1.3
- new net K4: DD113.PB0(ICP), DD3011.1.4
- new net K5: DD113.PB4(MISO), DD3011.2.1
- new net K6: DD113.PB5(SCK), DD113.PB6(XTAL1/TOSC1), DD3011.2.2
- new net K7: DD3011.2.3
- new net K8: DD113.PB7(XTAL2/TOSC2), DD3011.2.4
- new net K9: DD113.PC5(ADC5/SCL), DD3011.2.16
- new net N$32: IC1A.QD, IC1B.A
- new net N$35: DD113.PD3(INT1), KB.2, R106.1
- new net N$39: DD113.PD6(AIN0), KB.1, R105.1
- new net N$40: DD107C.O, DD107D.I0, DD107D.I1
- new net R: DD3011.1.10
- new net RES: DD3011.2.6
- new net SND: DD3011.1.12
- new net U7: DD107D.O, DD113.PD2(INT0)
- net +5V: now also DD113.AVCC, DD113.VCC@1, DD113.VCC@2, DD3011.2.15, KB.3, R105.2, R106.2
- net A0: now also DD3011.1.9
- net A1: now also DD3011.1.8
- net GND: now also DD113.GND, DD113.GND@1, DD113.GND@2, DD3011.1.7, KB.4
Other:
- note added: "40 39 38 37 36 35 34 33 32 31 30 29 28 27 26 25 24 23 22 21"
- note added: "Плата расширения DD101,DD104 КР565РУ5 DD105,DD108 К555ИР22 DD106,DD109 К555ИР16 DD107,DD110 К555ЛЕ1 DD111,DD112 К580ВВ55 DD113,DD114 ATMega8"
- note removed: "Плата расширения DD101,DD104 КР565РУ5 DD105,DD108 К555ИР22 DD106,DD109 К555ИР16 DD107,DD110 К155ЛЕ1 DD111,DD112 К580ВВ55 DD113,DD114 ATMega8"
- moved on the sheet: DD101, DD108, DD110B, DD113, DD113P

Commit message: v
Parts:
- added DD318.1, DD318.2: (no value), Разъёмы штырьковые 2.54мм:PINHD-1X12
Connections:
- new net B0: DD104.DO
- new net G0: DD103.DO
- new net N$42: DD110B.I1, DD110C.I1, DD110D.I1
- new net P1: DD112A.PA0
- new net P10: DD112A.PB1
- new net P11: DD112A.PB2
- new net P12: DD112A.PB3
- new net P13: DD112A.PB4
- new net P14: DD112A.PB5
- new net P15: DD112A.PB6
- new net P16: DD112A.PB7
- new net P2: DD112A.PA1
- new net P3: DD112A.PA2
- new net P4: DD112A.PA3
- new net P5: DD112A.PA4
- new net P6: DD112A.PA5
- new net P7: DD112A.PA6
- new net P8: DD112A.PA7
- new net P9: DD112A.PB0
- new net R0: DD102.DO
- new net R1: DD318.1.2, DD318.2.11
- new net VD0: DD318.1.4
- new net VD1: DD318.1.6
- new net VD2: DD318.1.8
- new net VD3: DD318.1.10
- new net VD4: DD318.2.10
- new net VD5: DD318.2.8
- new net VD6: DD318.2.6
- new net VD7: DD318.2.4
- net !CAS: now also DD102.!CAS, DD103.!CAS, DD104.!CAS
- net !RAS: now also DD102.!RAS, DD103.!RAS, DD104.!RAS, DD318.1.1
- net !WE: now also DD102.!WE, DD103.!WE, DD104.!WE
- net +5V: now also DD114.AVCC, DD114.VCC@1, DD114.VCC@2, DD318.2.1
- net B: now also DD104.DI
- net G: now also DD103.DI
- net G19: now also DD318.2.12
- net GND: now also DD114.GND, DD114.GND@1, DD114.GND@2, DD318.1.11, DD318.1.12
- net MA0: now also DD102.A0, DD103.A0, DD104.A0
- net MA1: now also DD102.A1, DD103.A1, DD104.A1
- net MA2: now also DD102.A2, DD103.A2, DD104.A2
- net MA3: now also DD102.A3, DD103.A3, DD104.A3
- net MA4: now also DD102.A4, DD103.A4, DD104.A4
- net MA5: now also DD102.A5, DD103.A5, DD104.A5
- net MA6: now also DD102.A6, DD103.A6, DD104.A6
- net MA7: now also DD102.A7, DD103.A7, DD104.A7
- net MD0: now also DD318.1.3
- net MD1: now also DD318.1.5
- net MD2: now also DD318.1.7
- net MD3: now also DD318.1.9
- net MD4: now also DD318.2.9
- net MD5: now also DD318.2.7
- net MD6: now also DD318.2.5
- net MD7: now also DD318.2.3
- net R: now also DD102.DI
Other:
- note added: "* есть"
- note added: "24 23 22 21 20 19 18 17 15 15 14 13"
- moved on the sheet: DD101, DD103, DD104, DD105, DD106, DD107C, DD107D, DD107P, DD108, DD109, DD112, DD113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

Commit message: .
Parts:
- removed DD101: КР565РУ5, ic-package:DIL16
- DD39: value (none) -> К573РФ4
Connections:
- new net CRG: DD105A.ENC, DD107A.O
- new net N$44: DD107A.I1, DD107B.O
- net !RAS: now also DD107A.I0
- net G19: now also DD107B.I0, DD107B.I1
- net GND: now also DD105A.OC
- net MD0: now also DD105A.1D
- net MD1: now also DD105A.2D
- net MD2: now also DD105A.3D
- net MD3: now also DD105A.4D
- net MD4: now also DD105A.5D
- net MD5: now also DD105A.6D
- net MD6: now also DD105A.7D
- net MD7: now also DD105A.8D
- net VD0: now also DD105A.1Q
- net VD1: now also DD105A.2Q
- net VD2: now also DD105A.3Q
- net VD3: now also DD105A.4Q
- net VD4: now also DD105A.5Q
- net VD5: now also DD105A.6Q
- net VD6: now also DD105A.7Q
- net VD7: now also DD105A.8Q
Other:
- note added: "DD1 использован DD21"

Commit message: d
Parts:
- removed DD106: К555ИР16, 74xx-eu:7495N
- removed DD113P: MEGA8-P, atmel:MEGA8-P
- added DD336.1, DD336.2: (no value), Разъёмы штырьковые 2.54мм:PINHD-1X7
- added LED1: (no value), led:LED5MM
- added R107: 560, rcl:R-EU_M0805
- added R7, R8, R9: (no value), rcl:R-TRIMM3296W
Connections:
- new net CLK: DD109A.CK1, DD336.2.6
- new net LED: DD114.PB0(ICP), R107.1
- new net N$43: DD108A.1Q, DD109A.A
- new net N$45: DD108A.2Q, DD109A.B
- new net N$46: DD108A.3Q, DD109A.C
- new net N$48: LED1.A, R107.2
- new net N$50: DD109A.QA, DD110B.I0
- new net N$51: DD109A.QB, DD110C.I0
- new net N$52: DD109A.QC, DD110D.I0
- new net N$54: DD110B.O, R7.A
- new net N$55: DD110C.O, R8.A
- new net N$56: DD110D.O, R9.A
- new net N$58: R7.S
- new net N$59: R8.S
- new net N$60: R9.S
- new net P17: DD112A.PC0
- new net P18: DD112A.PC1
- new net P19: DD112A.PC2
- new net P20: DD112A.PC3
- new net P21: DD112A.PC4
- new net P22: DD112A.PC5
- new net P23: DD112A.PC6
- new net P24: DD112A.PC7
- new net Q3: DD109A.MOD, DD336.1.6
- new net R2: DD109A.CK2, DD109A.SER, DD336.2.7
- new net SH: DD336.1.1
- new net VD10: DD336.1.4
- new net VD11: DD336.1.5
- new net VD8: DD336.1.2
- new net VD9: DD336.1.3
- new net VID: DD110A.I0, DD110A.I1, DD336.2.5
- net +5V: now also DD105P.VCC, DD107P.VCC, DD108P.VCC, DD109P.VCC, DD110P.VCC, DD336.2.1
- net B0: now also DD108A.3D
- net CRG: now also DD108A.ENC
- net G0: now also DD108A.2D
- net GND: now also DD105P.GND, DD107P.GND, DD108A.4D, DD108A.5D, DD108A.6D, DD108A.7D, DD108A.8D, DD108A.OC, DD108P.GND, DD109A.D, DD109P.GND, DD110P.GND, DD336.1.7, LED1.C, R7.E, R8.E, R9.E
- net N$42: now also DD110A.O
- net P16: now also DD114.PC0(ADC0)
- net R0: now also DD108A.1D
Other:
- note added: "14 13 12 11 10 9 8"
- note added: "24 23 22 21 20 19 18 17 16 15 14 13"
- note added: "DD1 использован DD28"
- note added: "DD6 использован DD33"
- note removed: "24 23 22 21 20 19 18 17 15 15 14 13"
- note removed: "DD1 использован DD21"
- moved on the sheet: DD102, DD103, DD104, DD105, DD107A, DD107B, DD107C, DD107D, DD107P, DD108, DD108P, DD109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

Commit message: .
Parts:
- removed DD105: К555ИР22, 74xx-eu:74LS373N
- removed DD49.2, DD50.2: К589АП16, ic-package:DIL16
- added 27512: (no value), memory:27512
- added DD31-: К589ИР12, 589:589IR12
- added IC2: (no value), ic-package:DIL24-6
- added R15, R23: 2k, rcl:R-EU_M1206
- DD31: value К589ИР12 -> К555ИР22; device 589:589IR12 -> 74xx-eu:74LS373N
Connections:
- removed net N$30: DD1A.O
- new net N$49: DD32A.CK2, DD33A.CK2, R23.1
- new net N$53: DD32A.CK1, DD33A.CK1, DD9F.O
- new net N$57: DD32A.MOD, DD33A.MOD, DD9B.O
- net !CAS: now also DD1A.O
- net !RAS: now also DD7C.O, IC2.1
- net +5V: now also DD31P.VCC, IC2.24, R15.2, R23.2; no longer DD105P.VCC
- net CRG: now also DD31A.ENC; no longer DD105A.ENC
- net G19: now also IC2.13
- net GND: now also DD31A.OC, DD31P.GND, DD32A.SER, IC2.11, IC2.12; no longer DD105A.OC, DD105P.GND
- net MD0: now also DD31A.1D, IC2.3; no longer DD105A.1D
- net MD1: now also DD31A.2D, IC2.5; no longer DD105A.2D
- net MD2: now also DD31A.3D, IC2.7; no longer DD105A.3D
- net MD3: now also DD31A.4D, IC2.9; no longer DD105A.4D
- net MD4: now also DD31A.5D, IC2.16; no longer DD105A.5D
- net MD5: now also DD31A.6D, IC2.18; no longer DD105A.6D
- net MD6: now also DD31A.7D, IC2.20; no longer DD105A.7D
- net MD7: now also DD31A.8D, IC2.22; no longer DD105A.8D
- net N$28: now also DD32A.QD, DD33A.SER; no longer C10.+, C11.1, R4.2
- net R1: now also IC2.14, IC2.2, R15.1
- net VD0: now also DD31A.1Q, DD32A.A, IC2.4; no longer DD105A.1Q
- net VD1: now also DD31A.2Q, DD32A.B, IC2.6; no longer DD105A.2Q
- net VD2: now also DD31A.3Q, DD32A.C, IC2.8; no longer DD105A.3Q
- net VD3: now also DD31A.4Q, DD32A.D, IC2.10; no longer DD105A.4Q
- net VD4: now also DD31A.5Q, DD33A.A, IC2.15; no longer DD105A.5Q
- net VD5: now also DD31A.6Q, DD33A.B, IC2.17; no longer DD105A.6Q
- net VD6: now also DD31A.7Q, DD33A.C, IC2.19; no longer DD105A.7Q
- net VD7: now also DD31A.8Q, DD33A.D, IC2.21; no longer DD105A.8Q
- net VID: now also C10.+, C11.1, DD33A.QD, R4.2
Other:
- moved on the sheet: DD14D, DD19, DD32, DD33, R47, R48

Commit message: -b
Parts:
- added JP2: (no value), Разъёмы штырьковые 2.54мм:PINHD-2X13
Connections:
- new net !U6: DD112A.CS
Changed lines of the file:
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@@
 <setting verticaltext="up"/>
 </settings>
-<grid distance="100" unitdist="mil" unit="mil" style="lines" multiple="1" display="yes" altdistance="0.01" altunitdist="inch" altunit="inch"/>
+<grid distance="0.1" unitdist="inch" unit="inch" style="lines" multiple="1" display="yes" altdistance="0.01" altunitdist="inch" altunit="inch"/>
 <layers>
 <layer number="1" name="Top" color="4" fill="1" visible="no" active="no"/>
@@
 <part name="R23" library="rcl" deviceset="R-EU_" device="M1206" value="2k"/>
 <part name="P+30" library="supply1" deviceset="+5V" device=""/>
+<part name="JP2" library="Разъёмы штырьковые 2.54мм" deviceset="PINHD-2X13" device=""/>
 </parts>
 <sheets>
@@
 <attribute name="VALUE" x="337.82" y="251.46" size="1.778" layer="96" rot="R180"/>
 </instance>
+<instance part="JP2" gate="A" x="-119.38" y="292.1"/>
 </instances>
 <busses>
@@
 </segment>
 </bus>
-<bus name="A[0..10],A'[11..15],D[0..7],G[1..19],MA[0..7],MD[0..7],VD[0..11],!RAS,!CAS,CLK,!WE,X-----X,K[1..27],U7,!U7,!WR,!RESIN,RES,!RD,B,G,R,B0,G0,R0,SND,VID,LED,P[1..24],R1,R2,CRG,SH,Q3">
+<bus name="A[0..10],A'[11..15],D[0..7],G[1..19],MA[0..7],MD[0..7],VD[0..11],!RAS,!CAS,CLK,!WE">
 <segment>
 <wire x1="322.58" y1="254" x2="322.58" y2="187.96" width="0.762" layer="92"/>
@@
 </instances>
 <busses>
-<bus name="A[0..10],A'[11..15],D[0..7],G[1..19],MA[0..7],MD[0..7],VD[0..11],!RAS,!CAS,CLK,!WE,X-----X,K[1..27],U7,!U7,!WR,!RESIN,RES,!RD,B,G,R,B0,G0,R0,SND,VID,LED,P[1..24],R1,R2,CRG,SH,Q3">
+<bus name="A[0..10],A'[11..15],D[0..7],G[1..19],MA[0..7],MD[0..7],VD[0..11],!RAS,!CAS,CLK,!WE,X-----X,K[1..27],U7,!U6,!U7,!WR,!RESIN,RES,!RD,B,G,R,B0,G0,R0,SND,VID,LED,P[1..24],R1,R2,CRG,SH,Q3">
 <segment>
 <wire x1="60.96" y1="40.64" x2="35.56" y2="40.64" width="0.762" layer="92"/>
@@
 </segment>
 </net>
+<net name="!U6" class="0">
+<segment>
+<pinref part="DD112" gate="A" pin="CS"/>
+<wire x1="223.52" y1="63.5" x2="233.68" y2="63.5" width="0.1524" layer="91"/>
+</segment>
+</net>

Commit message: s
Parts:
- removed DD54.1: К580ВА86, ic-package:DIL20
- removed DD55.1, DD56.1: К580ИР82, ic-package:DIL20
- removed IC2: (no value), ic-package:DIL24-6
- removed JP2: (no value), Разъёмы штырьковые 2.54мм:PINHD-2X13
- removed R15: 2k, rcl:R-EU_M1206
Connections:
- net !RAS: no longer IC2.1
- net +5V: no longer IC2.24, R15.2
- net G19: no longer IC2.13
- net GND: no longer IC2.11, IC2.12
- net MD0: no longer IC2.3
- net MD1: no longer IC2.5
- net MD2: no longer IC2.7
- net MD3: no longer IC2.9
- net MD4: no longer IC2.16
- net MD5: no longer IC2.18
- net MD6: no longer IC2.20
- net MD7: no longer IC2.22
- net R1: no longer IC2.14, IC2.2, R15.1
- net VD0: no longer IC2.4
- net VD1: no longer IC2.6
- net VD2: no longer IC2.8
- net VD3: no longer IC2.10
- net VD4: no longer IC2.15
- net VD5: no longer IC2.17
- net VD6: no longer IC2.19
- net VD7: no longer IC2.21
