File: SpecialistEE20.sch (EAGLE design)
At the start: 101 parts, among them IC1 74393N

Commit message: .
Parts:
- DD45: value 74393N -> К555ИЕ19
- renumbered IC1 to DD45
Connections:
- new net N$30: DD45A.QA
- new net N$47: DD45A.QB
- new net N$61: DD45A.QC
- new net N$62: DD45B.QA
- new net N$63: DD45B.QB
- new net N$64: DD45A.A
- new net N$65: DD45A.CLR, DD45B.CLR
- net D0: now also DD112A.D0
- net D1: now also DD112A.D1
- net D2: now also DD112A.D2
- net D3: now also DD112A.D3
- net D4: now also DD112A.D4
- net D5: now also DD112A.D5
- net D6: now also DD112A.D6
- net D7: now also DD112A.D7
Other:
- moved on the sheet: LED1, R107
Changed lines of the file:
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@@
 <part name="DD3011.2" library="Разъёмы штырьковые 2.54мм" deviceset="PINHD-1X20" device=""/>
 <part name="KB" library="Speccy" deviceset="MINI-DIN6" device="PTH" value="MINI-DIN6"/>
-<part name="IC1" library="74xx-eu" deviceset="74*393" device="N"/>
+<part name="DD45" library="74xx-eu" deviceset="74*393" device="N" value="К555ИЕ19"/>
 <part name="R105" library="rcl" deviceset="R-EU_" device="M0805" value="4k7"/>
 <part name="R106" library="rcl" deviceset="R-EU_" device="M0805" value="4k7"/>
@@
 </instance>
 <instance part="GND22" gate="1" x="368.3" y="-81.28"/>
-<instance part="IC1" gate="A" x="-35.56" y="142.24"/>
-<instance part="IC1" gate="B" x="-35.56" y="116.84"/>
+<instance part="DD45" gate="A" x="-35.56" y="142.24"/>
+<instance part="DD45" gate="B" x="-35.56" y="116.84"/>
 <instance part="27512" gate="A" x="408.94" y="-154.94"/>
 <instance part="DD31" gate="A" x="294.64" y="233.68"/>
@@
 <wire x1="48.26" y1="213.36" x2="48.26" y2="33.02" width="0.762" layer="92"/>
 <wire x1="48.26" y1="33.02" x2="73.66" y2="33.02" width="0.762" layer="92"/>
-</segment>
-<segment>
 <wire x1="322.58" y1="254" x2="322.58" y2="187.96" width="0.762" layer="92"/>
 <wire x1="322.58" y1="254" x2="375.92" y2="254" width="0.762" layer="92"/>
@@
 <wire x1="271.78" y1="254" x2="271.78" y2="218.44" width="0.762" layer="92"/>
 <wire x1="271.78" y1="254" x2="246.38" y2="254" width="0.762" layer="92"/>
-<wire x1="246.38" y1="254" x2="246.38" y2="205.74" width="0.762" layer="92"/>
+<wire x1="246.38" y1="254" x2="246.38" y2="198.12" width="0.762" layer="92"/>
 <wire x1="322.58" y1="254" x2="317.5" y2="254" width="0.762" layer="92"/>
+<wire x1="180.34" y1="198.12" x2="246.38" y2="198.12" width="0.762" layer="92"/>
 </segment>
 <segment>
@@
 <net name="N$32" class="0">
 <segment>
-<pinref part="IC1" gate="A" pin="QD"/>
+<pinref part="DD45" gate="A" pin="QD"/>
 <wire x1="-22.86" y1="137.16" x2="-20.32" y2="137.16" width="0.1524" layer="91"/>
 <wire x1="-20.32" y1="137.16" x2="-20.32" y2="129.54" width="0.1524" layer="91"/>
 <wire x1="-20.32" y1="129.54" x2="-50.8" y2="129.54" width="0.1524" layer="91"/>
 <wire x1="-50.8" y1="129.54" x2="-50.8" y2="119.38" width="0.1524" layer="91"/>
-<pinref part="IC1" gate="B" pin="A"/>
+<pinref part="DD45" gate="B" pin="A"/>
 <wire x1="-50.8" y1="119.38" x2="-48.26" y2="119.38" width="0.1524" layer="91"/>
+<wire x1="-20.32" y1="137.16" x2="-12.7" y2="137.16" width="0.1524" layer="91"/>
+<junction x="-20.32" y="137.16"/>
 </segment>
 </net>
@@
 </segment>
 </net>
+<net name="N$30" class="0">
+<segment>
+<pinref part="DD45" gate="A" pin="QA"/>
+<wire x1="-22.86" y1="144.78" x2="-12.7" y2="144.78" width="0.1524" layer="91"/>
+</segment>
+</net>
+<net name="N$47" class="0">
+<segment>
+<pinref part="DD45" gate="A" pin="QB"/>
+<wire x1="-22.86" y1="142.24" x2="-12.7" y2="142.24" width="0.1524" layer="91"/>
+</segment>
+</net>
+<net name="N$61" class="0">
+<segment>
+<pinref part="DD45" gate="A" pin="QC"/>
+<wire x1="-22.86" y1="139.7" x2="-12.7" y2="139.7" width="0.1524" layer="91"/>
+</segment>
+</net>
+<net name="N$62" class="0">
+<segment>
+<pinref part="DD45" gate="B" pin="QA"/>
+<wire x1="-22.86" y1="119.38" x2="-12.7" y2="119.38" width="0.1524" layer="91"/>
+</segment>
+</net>
+<net name="N$63" class="0">
+<segment>
+<pinref part="DD45" gate="B" pin="QB"/>
+<wire x1="-22.86" y1="116.84" x2="-12.7" y2="116.84" width="0.1524" layer="91"/>
+</segment>
+</net>
+<net name="N$64" class="0">
+<segment>
+<pinref part="DD45" gate="A" pin="A"/>
+<wire x1="-48.26" y1="144.78" x2="-50.8" y2="144.78" width="0.1524" layer="91"/>
+<wire x1="-50.8" y1="144.78" x2="-50.8" y2="152.4" width="0.1524" layer="91"/>
+<wire x1="-50.8" y1="152.4" x2="-12.7" y2="152.4" width="0.1524" layer="91"/>
+</segment>
+</net>
+<net name="N$65" class="0">
+<segment>
+<pinref part="DD45" gate="A" pin="CLR"/>
+<wire x1="-48.26" y1="137.16" x2="-53.34" y2="137.16" width="0.1524" layer="91"/>
+<wire x1="-53.34" y1="137.16" x2="-53.34" y2="111.76" width="0.1524" layer="91"/>
+<pinref part="DD45" gate="B" pin="CLR"/>
+<wire x1="-53.34" y1="111.76" x2="-48.26" y2="111.76" width="0.1524" layer="91"/>
+</segment>
+</net>
 </nets>
 </sheet>
@@
 <instance part="R9" gate="G$1" x="187.96" y="195.58" rot="R270"/>
 <instance part="GND36" gate="1" x="195.58" y="190.5"/>
-<instance part="LED1" gate="G$1" x="360.68" y="60.96"/>
-<instance part="R107" gate="G$1" x="353.06" y="66.04"/>
-<instance part="GND37" gate="1" x="360.68" y="50.8"/>
+<instance part="LED1" gate="G$1" x="358.14" y="60.96"/>
+<instance part="R107" gate="G$1" x="350.52" y="66.04"/>
+<instance part="GND37" gate="1" x="358.14" y="50.8"/>
 </instances>
 <busses>
@@
 <wire x1="246.38" y1="193.04" x2="223.52" y2="193.04" width="0.762" layer="92"/>
 <wire x1="223.52" y1="193.04" x2="223.52" y2="63.5" width="0.762" layer="92"/>
-<wire x1="342.9" y1="193.04" x2="342.9" y2="48.26" width="0.762" layer="92"/>
+<wire x1="342.9" y1="193.04" x2="342.9" y2="53.34" width="0.762" layer="92"/>
 </segment>
 <segment>
@@
 <pinref part="LED1" gate="G$1" pin="C"/>
 <pinref part="GND37" gate="1" pin="GND"/>
-<wire x1="360.68" y1="53.34" x2="360.68" y2="55.88" width="0.1524" layer="91"/>
+<wire x1="358.14" y1="53.34" x2="358.14" y2="55.88" width="0.1524" layer="91"/>
 </segment>
 </net>
@@
 <label x="264.16" y="170.18" size="1.778" layer="95"/>
 </segment>
+<segment>
+<pinref part="DD112" gate="A" pin="D0"/>
+<wire x1="223.52" y1="111.76" x2="233.68" y2="111.76" width="0.1524" layer="91"/>
+<label x="226.06" y="111.76" size="1.778" layer="95"/>
+</segment>
 </net>
 <net name="D1" class="0">
@@
 <label x="264.16" y="167.64" size="1.778" layer="95"/>
 </segment>
+<segment>
+<pinref part="DD112" gate="A" pin="D1"/>
+<wire x1="223.52" y1="109.22" x2="233.68" y2="109.22" width="0.1524" layer="91"/>
+<label x="226.06" y="109.22" size="1.778" layer="95"/>
+</segment>
 </net>
 <net name="D2" class="0">
@@
 <label x="264.16" y="165.1" size="1.778" layer="95"/>
 </segment>
+<segment>
+<pinref part="DD112" gate="A" pin="D2"/>
+<wire x1="223.52" y1="106.68" x2="233.68" y2="106.68" width="0.1524" layer="91"/>
+<label x="226.06" y="106.68" size="1.778" layer="95"/>
+</segment>
 </net>
 <net name="D3" class="0">
@@
 <label x="264.16" y="162.56" size="1.778" layer="95"/>
 </segment>
+<segment>
+<pinref part="DD112" gate="A" pin="D3"/>
+<wire x1="223.52" y1="104.14" x2="233.68" y2="104.14" width="0.1524" layer="91"/>
+<label x="226.06" y="104.14" size="1.778" layer="95"/>
+</segment>
 </net>
 <net name="D4" class="0">
@@
 <label x="264.16" y="160.02" size="1.778" layer="95"/>
 </segment>
+<segment>
+<pinref part="DD112" gate="A" pin="D4"/>
+<wire x1="223.52" y1="101.6" x2="233.68" y2="101.6" width="0.1524" layer="91"/>
+<label x="226.06" y="101.6" size="1.778" layer="95"/>
+</segment>
 </net>
 <net name="D5" class="0">
@@
 <label x="264.16" y="157.48" size="1.778" layer="95"/>
 </segment>
+<segment>
+<pinref part="DD112" gate="A" pin="D5"/>
+<wire x1="223.52" y1="99.06" x2="233.68" y2="99.06" width="0.1524" layer="91"/>
+<label x="226.06" y="99.06" size="1.778" layer="95"/>
+</segment>
 </net>
 <net name="D6" class="0">
@@
 <label x="264.16" y="154.94" size="1.778" layer="95"/>
 </segment>
+<segment>
+<pinref part="DD112" gate="A" pin="D6"/>
+<wire x1="223.52" y1="96.52" x2="233.68" y2="96.52" width="0.1524" layer="91"/>
+<label x="226.06" y="96.52" size="1.778" layer="95"/>
+</segment>
 </net>
 <net name="D7" class="0">
@@
 <label x="264.16" y="152.4" size="1.778" layer="95"/>
 </segment>
+<segment>
+<pinref part="DD112" gate="A" pin="D7"/>
+<wire x1="223.52" y1="93.98" x2="233.68" y2="93.98" width="0.1524" layer="91"/>
+<label x="226.06" y="93.98" size="1.778" layer="95"/>
+</segment>
 </net>
 <net name="K27" class="0">
@@
 <pinref part="DD114" gate="G$1" pin="PB0(ICP)"/>
 <pinref part="R107" gate="G$1" pin="1"/>
-<wire x1="332.74" y1="66.04" x2="347.98" y2="66.04" width="0.1524" layer="91"/>
+<wire x1="332.74" y1="66.04" x2="345.44" y2="66.04" width="0.1524" layer="91"/>
 <label x="335.28" y="66.04" size="1.778" layer="95"/>
 </segment>
@@
 <segment>
 <pinref part="R107" gate="G$1" pin="2"/>
-<wire x1="358.14" y1="66.04" x2="360.68" y2="66.04" width="0.1524" layer="91"/>
+<wire x1="355.6" y1="66.04" x2="358.14" y2="66.04" width="0.1524" layer="91"/>
 <pinref part="LED1" gate="G$1" pin="A"/>
-<wire x1="360.68" y1="66.04" x2="360.68" y2="63.5" width="0.1524" layer="91"/>
+<wire x1="358.14" y1="66.04" x2="358.14" y2="63.5" width="0.1524" layer="91"/>
 </segment>
 </net>

Commit message: d
Parts:
- removed DD31-: К589ИР12, 589:589IR12
Other:
- note added: "Новый (для оригинала) DD1 К555ЛН1 DD2,DD8 К555ИЕ7 DD3-DD5 К555ИЕ5 DD6 К555ЛЕ1 DD7 К555ЛА4 DD10 К555ЛА2 DD11,DD14 К555ЛА3 DD12 К555ТМ2 DD15-DD18 К555КП2 DD19 К155ЛП10 DD20 К155ЛА8 DD21-DD28 КР565РУ5 DD29 КР580ВМ80 DD30 К580ВВ55 DD31 К589ИР12 DD32,DD33 К555ИР16(К155ИР1) DD34(DD34,DD35) К555АП6 DD36, DD40 К555ИД4 DD37,DD38 К573РФ2 DD39 К573РФ4 DA1 КР544УД2"
- note added: "Этот вариант DD1 К555ЛН1 DD2,DD8 К555ИЕ7 DD3-DD5 К555ИЕ5 DD6,DD107,DD110 К555ЛЕ1 DD7 К555ЛА4 DD10 К555ЛА2 DD11,DD14 К555ЛА3 DD12 К555ТМ2 DD15-DD18 К555КП2 DD19 К555АП4 DD20 К155ЛА8 DD21-DD28,DD102-DD104 КР565РУ5 DD29 КР580ВМ80 DD30,DD112 К580ВВ55 DD31,DD108 К555ИР22 DD32,DD33,DD109 К555ИР16 DD34 К555АП6 DD36, DD40 К555ИД4 DD37,DD38 К573РФ2 DD39 К573РФ4 DD113,DD114 ATMega8 DA1 КР544УД2"
- note removed: "Новый (для оригинала) DD1 К555ЛН1 DD2,DD8 К555ИЕ7 DD3-DD5 К555ИЕ5 DD6 К555ЛЕ1 DD7 К555ЛА4 DD10 К555ЛА2 DD11,DD14 К555ЛА3 DD12 К555ТМ2 DD15-DD18 К555КП2 DD19 К155ЛП10 DD20 К155ЛА8 DD21-DD28 КР565РУ5 DD29 КР580ВМ80 DD30 К580ВВ55 DD31 К589ИР12 DD32,DD33 К555ИР16(К155ИР1)*295(*95) DD34(DD34,DD35) К555АП6 DD36, DD40 К555ИД4 DD37,DD38 К573РФ2 DD39 К573РФ4 DA1 КР544УД2"
Changed lines of the file:
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@@
 <part name="P+9" library="supply1" deviceset="+5V" device=""/>
 <part name="RD2" library="rcl" deviceset="R-EU_" device="M1206" value="2k"/>
-<part name="DD31-" library="589" deviceset="589IR12" device="" value="К589ИР12"/>
 <part name="DD28" library="memory" deviceset="2164" device="" value="КР565РУ5"/>
 <part name="DD22" library="memory" deviceset="2164" device="" value="КР565РУ5"/>
@@
 ТТЛ=1.1426 А
 +1323=2.4656 А</text>
-<text x="121.92" y="259.08" size="1.778" layer="98" rot="MR180">Новый
+<text x="119.38" y="259.08" size="1.778" layer="98" rot="MR180">Новый
 (для оригинала)
 DD1 К555ЛН1
@@
 DD30  К580ВВ55
 DD31 К589ИР12
-DD32,DD33 К555ИР16(К155ИР1)*295(*95)
+DD32,DD33 К555ИР16(К155ИР1)
 DD34(DD34,DD35) К555АП6
 DD36, DD40 К555ИД4
@@
 DA1 КР544УД2
 </text>
-<text x="121.92" y="180.34" size="1.778" layer="98" rot="MR180">Плата расширения
+<text x="119.38" y="182.88" size="1.778" layer="98" rot="MR180">Плата расширения
 DD101,DD104 КР565РУ5
 DD105,DD108 К555ИР22
@@
 DD111,DD112 К580ВВ55
 DD113,DD114 ATMega8</text>
-<text x="172.72" y="259.08" size="1.778" layer="98" rot="MR180">* есть
+<text x="218.44" y="259.08" size="1.778" layer="98" rot="MR180">* есть
 </text>
+<text x="160.02" y="259.08" size="1.778" layer="98" rot="MR180">Этот вариант
+DD1 К555ЛН1
+DD2,DD8 К555ИЕ7
+DD3-DD5 К555ИЕ5
+DD6,DD107,DD110  К555ЛЕ1
+DD7 К555ЛА4
+DD10 К555ЛА2
+DD11,DD14 К555ЛА3
+DD12 К555ТМ2
+DD15-DD18 К555КП2
+DD19 К555АП4
+DD20  К155ЛА8
+DD21-DD28,DD102-DD104 КР565РУ5
+DD29 КР580ВМ80
+DD30,DD112  К580ВВ55
+DD31,DD108 К555ИР22
+DD32,DD33,DD109 К555ИР16
+DD34 К555АП6
+DD36, DD40 К555ИД4
+DD37,DD38 К573РФ2
+DD39 К573РФ4
+DD113,DD114 ATMega8
+DA1 КР544УД2</text>
 </plain>
 <instances>
@@
 </instance>
 <instance part="RD2" gate="G$1" x="86.36" y="248.92"/>
-<instance part="DD31-" gate="P" x="187.96" y="-264.16"/>
 <instance part="DD28" gate="A" x="353.06" y="-60.96"/>
 <instance part="DD22" gate="A" x="78.74" y="-60.96"/>

Commit message: ..
Parts:
- added R14: 2k, rcl:R-EU_M1206
Connections:
- removed net CPU_F1: DD20C.O, R48.1
- removed net CPU_F2: DD20D.O, R47.1
- new net F1: DD20C.O, DD29.PHI1, R48.1
- new net F2: DD20D.O, DD29.PHI2, R47.1
- new net N$66: DD29.READY, R14.1
- new net RESET80: DD12A.!Q, DD29.RESET
- net !RD: now also DD112A.RD
- net +12V: now also DD29.VDD/+12V
- net +5V: now also DD29.VCC/+5V, R14.2
- net -5V: now also DD29.VBB/-5V
- net D0: now also DD29.D0
- net D1: now also DD29.D1
- net D2: now also DD29.D2
- net D3: now also DD29.D3
- net D4: now also DD29.D4
- net D5: now also DD29.D5
- net D6: now also DD29.D6
- net D7: now also DD29.D7
- net GND: now also DD29.INT, DD29.VSS/GND
- net RES: now also DD112A.RESET

Commit message: 8.
Connections:
- net RESET80 renamed RES80
- new net A11: DD29.A11
- new net A12: DD29.A12
- new net A13: DD29.A13
- new net A14: DD29.A14
- new net A15: DD29.A15
- net !WR: now also DD29.WR
- net A0: now also DD29.A0
- net A1: now also DD29.A1
- net A10: now also DD29.A10
- net A2: now also DD29.A2
- net A3: now also DD29.A3
- net A4: now also DD29.A4
- net A5: now also DD29.A5
- net A6: now also DD29.A6
- net A7: now also DD29.A7
- net A8: now also DD29.A8
- net A9: now also DD29.A9
- net GND: now also DD29.HOLD

Commit message: a
Parts:
- removed DD318.1, DD318.2: (no value), Разъёмы штырьковые 2.54мм:PINHD-1X12
Connections:
- removed net R1: DD318.1.2, DD318.2.11
- net !RAS: no longer DD318.1.1
- net +5V: now also DD32P.VCC, DD33P.VCC, DD34P.VCC, DD36P.VCC, DD40P.VCC; no longer DD318.2.1
- net G19: no longer DD318.2.12
- net GND: now also DD32P.GND, DD33P.GND, DD34P.GND, DD36P.GND, DD40P.GND; no longer DD318.1.11, DD318.1.12
- net MD0: no longer DD318.1.3
- net MD1: no longer DD318.1.5
- net MD2: no longer DD318.1.7
- net MD3: no longer DD318.1.9
- net MD4: no longer DD318.2.9
- net MD5: no longer DD318.2.7
- net MD6: no longer DD318.2.5
- net MD7: no longer DD318.2.3
- net VD0: no longer DD318.1.4
- net VD1: no longer DD318.1.6
- net VD2: no longer DD318.1.8
- net VD3: no longer DD318.1.10
- net VD4: no longer DD318.2.10
- net VD5: no longer DD318.2.8
- net VD6: no longer DD318.2.6
- net VD7: no longer DD318.2.4
Other:
- note removed: "24 23 22 21 20 19 18 17 16 15 14 13"
- moved on the sheet: DD107A, DD107B, DD31, DD32P, DD33P, DD40P

Commit message: o
Parts:
- added DD19': К555АП4, 74xx-eu:74LS241N
- added RD3: 2k, rcl:R-EU_M1206
Connections:
- new net N$67: DD19'B.G, RD3.2
- new net RD: DD29.DBIN
- net GND: now also DD19'A.G
Other:
- moved on the sheet: DD14D, DD19, DD30, DD32, DD33, DD336.1, DD336.2, DD34, R23

Commit message: ..
Other:
- moved on the sheet: 27512, DD39
Changed lines of the file:
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@@
 <instance part="DD33" gate="A" x="327.66" y="185.42"/>
 <instance part="DD38" gate="A" x="284.48" y="-177.8"/>
-<instance part="DD39" gate="A" x="355.6" y="-152.4"/>
+<instance part="DD39" gate="A" x="325.12" y="-129.54"/>
 <instance part="DD34" gate="A" x="266.7" y="147.32"/>
 <instance part="DD19" gate="A" x="464.82" y="172.72"/>
@@
 <instance part="DD45" gate="A" x="-35.56" y="142.24"/>
 <instance part="DD45" gate="B" x="-35.56" y="116.84"/>
-<instance part="27512" gate="A" x="408.94" y="-154.94"/>
+<instance part="27512" gate="A" x="368.3" y="-132.08"/>
 <instance part="DD31" gate="A" x="266.7" y="233.68"/>
 <instance part="GND31" gate="1" x="251.46" y="215.9"/>

Commit message: .
Parts:
- added DD13: К555ИР22, 74xx-eu:74LS373N
Connections:
- new net N$69: DD14A.O, DD34A.G
- new net N$70: DD12B.Q, DD14A.I1
- new net N$71: DD14A.I0
- net !RD: now also DD14D.O, DD34A.DIR
- net D0: now also DD34A.A1
- net D1: now also DD34A.A2
- net D2: now also DD34A.A8
- net D3: now also DD34A.A3
- net D4: now also DD34A.A4
- net D5: now also DD34A.A5
- net D6: now also DD34A.A6
- net D7: now also DD34A.A7
- net MD0: now also DD34A.B1
- net MD1: now also DD34A.B2
- net MD2: now also DD34A.B8
- net MD3: now also DD34A.B3
- net MD4: now also DD34A.B4
- net MD5: now also DD34A.B5
- net MD6: now also DD34A.B6
- net MD7: now also DD34A.B7
- net RD: now also DD14D.I0, DD14D.I1
