File: SpecialistEE20.sch (EAGLE design)
At the start: 102 parts

Commit message: 1
Other:
- moved on the sheet: DD14A
Changed lines of the file:
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@@
 <instance part="DD34" gate="P" x="210.82" y="-264.16"/>
 <instance part="DD36" gate="P" x="220.98" y="-264.16"/>
-<instance part="DD14" gate="A" x="259.08" y="104.14"/>
+<instance part="DD14" gate="A" x="259.08" y="101.6"/>
 <instance part="DD19'" gate="A" x="421.64" y="177.8"/>
 <instance part="DD19'" gate="B" x="421.64" y="152.4"/>
@@
 <wire x1="246.38" y1="134.62" x2="246.38" y2="127" width="0.1524" layer="91"/>
 <wire x1="246.38" y1="127" x2="271.78" y2="127" width="0.1524" layer="91"/>
-<wire x1="271.78" y1="127" x2="271.78" y2="104.14" width="0.1524" layer="91"/>
+<wire x1="271.78" y1="127" x2="271.78" y2="101.6" width="0.1524" layer="91"/>
 <pinref part="DD14" gate="A" pin="O"/>
-<wire x1="271.78" y1="104.14" x2="266.7" y2="104.14" width="0.1524" layer="91"/>
+<wire x1="271.78" y1="101.6" x2="266.7" y2="101.6" width="0.1524" layer="91"/>
 </segment>
 </net>
@@
 <wire x1="132.08" y1="5.08" x2="185.42" y2="5.08" width="0.1524" layer="91"/>
 <wire x1="185.42" y1="5.08" x2="185.42" y2="91.44" width="0.1524" layer="91"/>
-<wire x1="185.42" y1="91.44" x2="248.92" y2="91.44" width="0.1524" layer="91"/>
-<wire x1="248.92" y1="91.44" x2="248.92" y2="101.6" width="0.1524" layer="91"/>
+<wire x1="185.42" y1="91.44" x2="238.76" y2="91.44" width="0.1524" layer="91"/>
+<wire x1="238.76" y1="91.44" x2="238.76" y2="99.06" width="0.1524" layer="91"/>
 <pinref part="DD14" gate="A" pin="I1"/>
-<wire x1="248.92" y1="101.6" x2="251.46" y2="101.6" width="0.1524" layer="91"/>
+<wire x1="238.76" y1="99.06" x2="251.46" y2="99.06" width="0.1524" layer="91"/>
 </segment>
 </net>
@@
 <segment>
 <pinref part="DD14" gate="A" pin="I0"/>
-<wire x1="251.46" y1="106.68" x2="246.38" y2="106.68" width="0.1524" layer="91"/>
-<wire x1="246.38" y1="106.68" x2="246.38" y2="93.98" width="0.1524" layer="91"/>
-<wire x1="246.38" y1="93.98" x2="259.08" y2="93.98" width="0.1524" layer="91"/>
-</segment>
-</net>
+<wire x1="251.46" y1="104.14" x2="246.38" y2="104.14" width="0.1524" layer="91"/>
+<wire x1="246.38" y1="104.14" x2="246.38" y2="88.9" width="0.1524" layer="91"/>
+<wire x1="246.38" y1="88.9" x2="259.08" y2="88.9" width="0.1524" layer="91"/>
+</segment>
+</net>

Commit message: g
Connections:
- net N$44 renamed !G19B
- net N$70 renamed !G19A
- removed net N$36: DD12B.D
- new net SNY: DD12B.D, DD29.SYNC
Other:
- moved on the sheet: DD14A, DD37
Changed lines of the file:
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@@
 <instance part="GND32" gate="1" x="429.26" y="208.28"/>
 <instance part="GND41" gate="1" x="187.96" y="132.08" rot="R270"/>
-<instance part="DD14" gate="A" x="259.08" y="101.6"/>
+<instance part="DD14" gate="A" x="264.16" y="101.6"/>
 <instance part="DD19'" gate="A" x="421.64" y="177.8"/>
 <instance part="DD19'" gate="B" x="421.64" y="152.4"/>
@@
 </instances>
 <busses>
-<bus name="A[0..15],A'[11..15],D[0..7],F[1..2],G[1..19],MA[0..7],MD[0..7],VD[0..11],!RAS,!CAS,CLK,!WE,!WR,X-----X,K[1..27],U7,!,U[6..7],!RESIN,RES,RES80,RD,!RD,B,G,R,B0,G0,R0,SND,VID,LED,P[1..24],R[1..2],CRG,SH,Q3">
+<bus name="A[0..15],A'[11..15],D[0..7],F[1..2],G[1..19],!G19A,MA[0..7],MD[0..7],VD[0..11],!RAS,!CAS,CLK,!WE,!WR,X-----X,K[1..27],U7,!,U[6..7],!RESIN,RES,RES80,RD,!RD,SNY,B,G,R,B0,G0,R0,SND,VID,LED,P[1..24],R[1..2],CRG,SH,Q3">
 <segment>
 <wire x1="180.34" y1="198.12" x2="180.34" y2="43.18" width="0.762" layer="92"/>
@@
 <wire x1="210.82" y1="198.12" x2="210.82" y2="231.14" width="0.762" layer="92"/>
 <wire x1="241.3" y1="198.12" x2="241.3" y2="167.64" width="0.762" layer="92"/>
-<wire x1="241.3" y1="167.64" x2="241.3" y2="104.14" width="0.762" layer="92"/>
+<wire x1="241.3" y1="167.64" x2="241.3" y2="96.52" width="0.762" layer="92"/>
 <wire x1="241.3" y1="198.12" x2="241.3" y2="254" width="0.762" layer="92"/>
 <wire x1="294.64" y1="254" x2="294.64" y2="187.96" width="0.762" layer="92"/>
@@
 <wire x1="241.3" y1="167.64" x2="284.48" y2="167.64" width="0.762" layer="92"/>
 <wire x1="284.48" y1="167.64" x2="284.48" y2="142.24" width="0.762" layer="92"/>
+<wire x1="139.7" y1="20.32" x2="134.62" y2="20.32" width="0.762" layer="92"/>
+<wire x1="134.62" y1="20.32" x2="134.62" y2="86.36" width="0.762" layer="92"/>
 </segment>
 <segment>
@@
 </segment>
 </net>
-<net name="N$36" class="0">
-<segment>
-<pinref part="DD12" gate="B" pin="D"/>
-<wire x1="91.44" y1="73.66" x2="86.36" y2="73.66" width="0.1524" layer="91"/>
-<wire x1="86.36" y1="73.66" x2="86.36" y2="25.4" width="0.1524" layer="91"/>
-<wire x1="86.36" y1="25.4" x2="116.84" y2="25.4" width="0.1524" layer="91"/>
-</segment>
-</net>
 <net name="N$37" class="0">
 <segment>
@@
 <pinref part="DD12" gate="B" pin="!Q"/>
 <wire x1="139.7" y1="66.04" x2="116.84" y2="66.04" width="0.1524" layer="91"/>
-<label x="121.92" y="66.04" size="1.778" layer="95"/>
+<label x="116.84" y="66.04" size="1.778" layer="95"/>
 </segment>
 <segment>
@@
 </segment>
 </net>
-<net name="N$44" class="0">
+<net name="!G19B" class="0">
 <segment>
 <pinref part="DD107" gate="B" pin="O"/>
 <pinref part="DD107" gate="A" pin="I1"/>
 <wire x1="269.24" y1="203.2" x2="271.78" y2="203.2" width="0.1524" layer="91"/>
+<label x="266.7" y="193.04" size="1.778" layer="95"/>
 </segment>
 </net>
@@
 <pinref part="DD12" gate="A" pin="!Q"/>
 <wire x1="139.7" y1="43.18" x2="116.84" y2="43.18" width="0.1524" layer="91"/>
-<label x="121.92" y="43.18" size="1.778" layer="95"/>
+<label x="116.84" y="43.18" size="1.778" layer="95"/>
 </segment>
 </net>
@@
 <wire x1="248.92" y1="134.62" x2="246.38" y2="134.62" width="0.1524" layer="91"/>
 <wire x1="246.38" y1="134.62" x2="246.38" y2="127" width="0.1524" layer="91"/>
-<wire x1="246.38" y1="127" x2="271.78" y2="127" width="0.1524" layer="91"/>
-<wire x1="271.78" y1="127" x2="271.78" y2="101.6" width="0.1524" layer="91"/>
+<wire x1="246.38" y1="127" x2="274.32" y2="127" width="0.1524" layer="91"/>
+<wire x1="274.32" y1="127" x2="274.32" y2="101.6" width="0.1524" layer="91"/>
 <pinref part="DD14" gate="A" pin="O"/>
-<wire x1="271.78" y1="101.6" x2="266.7" y2="101.6" width="0.1524" layer="91"/>
+<wire x1="274.32" y1="101.6" x2="271.78" y2="101.6" width="0.1524" layer="91"/>
 </segment>
 </net>
-<net name="N$70" class="0">
+<net name="N$71" class="0">
 <segment>
-<pinref part="DD12" gate="B" pin="Q"/>
-<wire x1="116.84" y1="76.2" x2="132.08" y2="76.2" width="0.1524" layer="91"/>
-<wire x1="132.08" y1="76.2" x2="132.08" y2="5.08" width="0.1524" layer="91"/>
-<wire x1="132.08" y1="5.08" x2="185.42" y2="5.08" width="0.1524" layer="91"/>
-<wire x1="185.42" y1="5.08" x2="185.42" y2="91.44" width="0.1524" layer="91"/>
-<wire x1="185.42" y1="91.44" x2="238.76" y2="91.44" width="0.1524" layer="91"/>
-<wire x1="238.76" y1="91.44" x2="238.76" y2="99.06" width="0.1524" layer="91"/>
-<pinref part="DD14" gate="A" pin="I1"/>
-<wire x1="238.76" y1="99.06" x2="251.46" y2="99.06" width="0.1524" layer="91"/>
+<pinref part="DD14" gate="A" pin="I0"/>
+<wire x1="256.54" y1="104.14" x2="251.46" y2="104.14" width="0.1524" layer="91"/>
+<wire x1="251.46" y1="104.14" x2="251.46" y2="88.9" width="0.1524" layer="91"/>
+<wire x1="251.46" y1="88.9" x2="259.08" y2="88.9" width="0.1524" layer="91"/>
 </segment>
 </net>
-<net name="N$71" class="0">
+<net name="SNY" class="0">
 <segment>
-<pinref part="DD14" gate="A" pin="I0"/>
-<wire x1="251.46" y1="104.14" x2="246.38" y2="104.14" width="0.1524" layer="91"/>
-<wire x1="246.38" y1="104.14" x2="246.38" y2="88.9" width="0.1524" layer="91"/>
-<wire x1="246.38" y1="88.9" x2="259.08" y2="88.9" width="0.1524" layer="91"/>
+<pinref part="DD29" gate="G$1" pin="SYNC"/>
+<wire x1="241.3" y1="116.84" x2="231.14" y2="116.84" width="0.1524" layer="91"/>
+<label x="233.68" y="116.84" size="1.778" layer="95"/>
+</segment>
+<segment>
+<pinref part="DD12" gate="B" pin="D"/>
+<wire x1="91.44" y1="73.66" x2="86.36" y2="73.66" width="0.1524" layer="91"/>
+<wire x1="86.36" y1="73.66" x2="86.36" y2="25.4" width="0.1524" layer="91"/>
+<wire x1="86.36" y1="25.4" x2="134.62" y2="25.4" width="0.1524" layer="91"/>
+<label x="127" y="25.4" size="1.778" layer="95"/>
+</segment>
+</net>
+<net name="!G19A" class="0">
+<segment>
+<pinref part="DD12" gate="B" pin="Q"/>
+<wire x1="116.84" y1="76.2" x2="134.62" y2="76.2" width="0.1524" layer="91"/>
+<label x="127" y="76.2" size="1.778" layer="95"/>
+</segment>
+<segment>
+<pinref part="DD14" gate="A" pin="I1"/>
+<wire x1="241.3" y1="99.06" x2="256.54" y2="99.06" width="0.1524" layer="91"/>
+<label x="243.84" y="99.06" size="1.778" layer="95"/>
 </segment>
 </net>
@@
 </plain>
 <instances>
-<instance part="DD37" gate="A" x="287.02" y="170.18"/>
+<instance part="DD37" gate="A" x="284.48" y="160.02"/>
 <instance part="DD38" gate="A" x="284.48" y="111.76"/>
 <instance part="DD39" gate="A" x="325.12" y="160.02"/>
@@
 </instances>
 <busses>
-<bus name="A[0..15],A'[11..15],D[0..7],F[1..2],G[1..19],MA[0..7],MD[0..7],VD[0..11],!RAS,!CAS,CLK,!WE,!WR,X-----X,K[1..27],U7,!,U[6..7],!RESIN,RES,RES80,RD,!RD,B,G,R,B0,G0,R0,SND,VID,LED,P[1..24],R[1..2],CRG,SH,Q3">
+<bus name="A[0..15],A'[11..15],D[0..7],F[1..2],G[1..19],MA[0..7],MD[0..7],VD[0..11],!RAS,!CAS,CLK,!WE,!WR,X-----X,K[1..27],U7,!,U[6..7],!RESIN,RES,RES80,RD,!RD,SNY,B,G,R,B0,G0,R0,SND,VID,LED,P[1..24],R[1..2],CRG,SH,Q3">
 <segment>
 <wire x1="55.88" y1="248.92" x2="10.16" y2="248.92" width="0.762" layer="92"/>
@@
 </instances>
 <busses>
-<bus name="A[0..15],A'[11..15],D[0..7],F[1..2],G[1..19],MA[0..7],MD[0..7],VD[0..11],!RAS,!CAS,CLK,!WE,!WR,X-----X,K[1..27],U7,!,U[6..7],!RESIN,RES,RES80,RD,!RD,B,G,R,B0,G0,R0,SND,VID,LED,P[1..24],R[1..2],CRG,SH,Q3">
+<bus name="A[0..15],A'[11..15],D[0..7],F[1..2],G[1..19],MA[0..7],MD[0..7],VD[0..11],!RAS,!CAS,CLK,!WE,!WR,X-----X,K[1..27],U7,!,U[6..7],!RESIN,RES,RES80,RD,!RD,SNY,B,G,R,B0,G0,R0,SND,VID,LED,P[1..24],R[1..2],CRG,SH,Q3">
 <segment>
 <wire x1="193.04" y1="167.64" x2="121.92" y2="167.64" width="0.762" layer="92"/>

Commit message: .
Parts:
- removed DD336.1, DD336.2: (no value), Разъёмы штырьковые 2.54мм:PINHD-1X7
- added JP2: (no value), Разъёмы штырьковые 2.54мм:PINHD-1X30
- added JP3, JP4: (no value), Разъёмы штырьковые 2.54мм:PINHD-1X20
- added X1: SCART-F, con-hirschmann:SCART-F
- DD13: value К555ИР22 -> КР580ВВ55; device 74xx-eu:74LS373N -> micro-intel:8255A
Connections:
- removed net N$53: DD32A.CK1, DD33A.CK1, DD9F.O
- removed net N$57: DD32A.MOD, DD33A.MOD, DD9B.O
- removed net SH: DD336.1.1
- removed net VD10: DD336.1.4
- removed net VD11: DD336.1.5
- removed net VD8: DD336.1.2
- removed net VD9: DD336.1.3
- net +5V: no longer DD336.2.1
- net CLK: now also DD32A.CK1, DD33A.CK1, DD9F.O; no longer DD336.2.6
- net GND: no longer DD336.1.7
- net Q3: now also DD32A.MOD, DD33A.MOD, DD9B.O; no longer DD336.1.6
- net R2: no longer DD336.2.7
- net VID: no longer DD336.2.5
Other:
- note removed: "14 13 12 11 10 9 8"
- note removed: "DD6 использован DD33"

Commit message: 9
Parts:
- removed DD13: КР580ВВ55, micro-intel:8255A
- removed DD19': К555АП4, 74xx-eu:74LS241N
- removed JP2: (no value), Разъёмы штырьковые 2.54мм:PINHD-1X30
- removed JP3, JP4: (no value), Разъёмы штырьковые 2.54мм:PINHD-1X20
- removed R7, R8: (no value), rcl:R-TRIMM3296W
- removed RD3: 2k, rcl:R-EU_M1206
- added J1: (no value), Speccy:SDCARD
- added R101, R102, R103: (no value), rcl:R-TRIMM3296W
- added U$2: SWITCH9X4, ESR_NM8032:SWITCH9X4
- R9: value (none) -> 2k; device rcl:R-TRIMM3296W -> rcl:R-EU_M1206
Connections:
- removed net N$67: DD19'B.G, RD3.2
- new net !R: DD114.PC1(ADC1)
- new net CS: DD114.PB2(SS/OC1B)
- new net MISO: DD114.PB4(MISO)
- new net MOSI: DD114.PB3(MOSI/OC2)
- new net N$36: DD20A.I1
- new net N$44: DD11A.O, DD20A.I0
- new net N$53: DD20A.O, DD9C.I
- new net SCK: DD114.PB5(SCK)
- new net TON: DD114.PC2(ADC2)
- net !RESIN: now also DD114.PC6(/RESET)
- net !WR: now also DD112A.WR
- net +5V: now also R9.2; no longer R13.2
- net A0: now also DD112A.A0
- net A1: now also DD112A.A1
- net GND: now also R101.E, R102.E, R103.E; no longer DD19'A.G, R7.E, R8.E, R9.E
- net N$18: now also R9.1; no longer R13.1
- net N$54: now also R101.A; no longer R7.A
- net N$55: now also R102.A; no longer R8.A
- net N$56: now also R103.A; no longer R9.A
- net N$58: now also R101.S; no longer R7.S
- net N$59: now also R102.S; no longer R8.S
- net N$60: now also R103.S; no longer R9.S
- net P17: now also DD114.PD0(RXD)
- net P18: now also DD114.PD1(TXD)
- net P19: now also DD114.PD2(INT0)
- net P20: now also DD114.PD3(INT1)
- net P21: now also DD114.PD4(XCK/T0)
- net P22: now also DD114.PD5(T1)
- net P23: now also DD114.PD6(AIN0)
- net P24: now also DD114.PD7(AIN1)

Commit message: .
Connections:
- net N$36 renamed STRT
- removed net N$71: DD14A.I0
- new net DD9DD14: DD14A.I0, DD36A.1G, DD36A.2C, DD9C.O
- net +5V: now also R13.2
- net A11: now also DD36A.B
- net A12: now also DD36A.A
- net A13: now also DD36A.1C, DD36A.2G
- net A14: now also DD11A.I0
- net A15: now also DD11A.I1
- net N$53: now also R13.1
Other:
- moved on the sheet: R13
Changed lines of the file:
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@@
 <part name="U$2" library="ESR_NM8032" deviceset="SWITCH9X4" device=""/>
 <part name="R13" library="rcl" deviceset="R-EU_" device="M1206" value="2k"/>
+<part name="P+25" library="supply1v" deviceset="+5V" device=""/>
 </parts>
 <sheets>
@@
 </instances>
 <busses>
-<bus name="A[0..15],A'[11..15],D[0..7],F[1..2],G[1..19],!G19A,MA[0..7],MD[0..7],VD[0..11],!RAS,!CAS,CLK,!WE,!WR,X-----X,K[1..27],U7,!U[6..7],!RESIN,RES,RES80,RD,!RD,SNY,B,G,R,B0,G0,R0,SND,VID,LED,P[1..24],R[1..2],CRG,CS,!R,SH,TON,Q3,MOSI,MISO,SCK">
+<bus name="A[0..15],A'[11..15],D[0..7],F[1..2],G[1..19],!G19A,MA[0..7],MD[0..7],VD[0..11],!RAS,!CAS,CLK,!WE,!WR,X-----X,K[1..27],U7,!U[6..7],!RESIN,RES,RES80,RD,!RD,SNY,STRT,B,G,R,B0,G0,R0,SND,VID,LED,P[1..24],R[1..2],CRG,CS,!R,SH,TON,Q3,MOSI,MISO,SCK">
 <segment>
 <wire x1="180.34" y1="198.12" x2="180.34" y2="43.18" width="0.762" layer="92"/>
@@
 </segment>
 </net>
-<net name="N$71" class="0">
+<net name="DD9DD14" class="0">
 <segment>
 <pinref part="DD14" gate="A" pin="I0"/>
@@
 <wire x1="251.46" y1="104.14" x2="251.46" y2="88.9" width="0.1524" layer="91"/>
 <wire x1="251.46" y1="88.9" x2="259.08" y2="88.9" width="0.1524" layer="91"/>
+<label x="254" y="88.9" size="1.778" layer="95"/>
 </segment>
 </net>
@@
 </instances>
 <busses>
-<bus name="A[0..15],A'[11..15],D[0..7],F[1..2],G[1..19],!G19A,MA[0..7],MD[0..7],VD[0..11],!RAS,!CAS,CLK,!WE,!WR,X-----X,K[1..27],U7,!U[6..7],!RESIN,RES,RES80,RD,!RD,SNY,B,G,R,B0,G0,R0,SND,VID,LED,P[1..24],R[1..2],CRG,CS,!R,SH,TON,Q3,MOSI,MISO,SCK">
+<bus name="A[0..15],A'[11..15],D[0..7],F[1..2],G[1..19],!G19A,MA[0..7],MD[0..7],VD[0..11],!RAS,!CAS,CLK,!WE,!WR,X-----X,K[1..27],U7,!U[6..7],!RESIN,RES,RES80,RD,!RD,SNY,STRT,B,G,R,B0,G0,R0,SND,VID,LED,P[1..24],R[1..2],CRG,CS,!R,SH,TON,Q3,MOSI,MISO,SCK">
 <segment>
 <wire x1="193.04" y1="167.64" x2="121.92" y2="167.64" width="0.762" layer="92"/>
@@
 <instance part="DD20" gate="A" x="185.42" y="111.76"/>
 <instance part="DD9" gate="C" x="208.28" y="111.76"/>
-<instance part="R13" gate="G$1" x="190.5" y="132.08" rot="R90"/>
+<instance part="R13" gate="G$1" x="195.58" y="119.38" rot="R90"/>
+<instance part="P+25" gate="1" x="195.58" y="129.54"/>
 </instances>
 <busses>
-<bus name="A[0..15],A'[11..15],D[0..7],F[1..2],G[1..19],!G19A,MA[0..7],MD[0..7],VD[0..11],!RAS,!CAS,CLK,!WE,!WR,X-----X,K[1..27],U7,!U[6..7],!RESIN,RES,RES80,RD,!RD,SNY,B,G,R,B0,G0,R0,SND,VID,LED,P[1..24],R[1..2],CRG,CS,!R,SH,TON,Q3,MOSI,MISO,SCK">
+<bus name="A[0..15],A'[11..15],D[0..7],F[1..2],G[1..19],!G19A,MA[0..7],MD[0..7],VD[0..11],!RAS,!CAS,CLK,!WE,!WR,X-----X,K[1..27],U7,!U[6..7],!RESIN,RES,RES80,RD,!RD,SNY,STRT,B,G,R,B0,G0,R0,SND,VID,LED,P[1..24],R[1..2],CRG,CS,!R,SH,TON,Q3,MOSI,MISO,SCK">
 <segment>
 <wire x1="55.88" y1="248.92" x2="10.16" y2="248.92" width="0.762" layer="92"/>
@@
 <wire x1="101.6" y1="248.92" x2="101.6" y2="213.36" width="0.762" layer="92"/>
 <wire x1="101.6" y1="248.92" x2="147.32" y2="248.92" width="0.762" layer="92"/>
-<wire x1="147.32" y1="248.92" x2="147.32" y2="213.36" width="0.762" layer="92"/>
 <wire x1="147.32" y1="248.92" x2="193.04" y2="248.92" width="0.762" layer="92"/>
 <wire x1="193.04" y1="248.92" x2="193.04" y2="213.36" width="0.762" layer="92"/>
@@
 <wire x1="330.2" y1="248.92" x2="375.92" y2="248.92" width="0.762" layer="92"/>
 <wire x1="375.92" y1="248.92" x2="375.92" y2="213.36" width="0.762" layer="92"/>
+<wire x1="147.32" y1="248.92" x2="147.32" y2="167.64" width="0.762" layer="92"/>
+<wire x1="147.32" y1="167.64" x2="147.32" y2="96.52" width="0.762" layer="92"/>
+<wire x1="147.32" y1="167.64" x2="187.96" y2="167.64" width="0.762" layer="92"/>
+<wire x1="187.96" y1="167.64" x2="187.96" y2="144.78" width="0.762" layer="92"/>
 </segment>
 </bus>
@@
 <pinref part="DD28" gate="A" pin="VCC"/>
 </segment>
+<segment>
+<pinref part="P+25" gate="1" pin="+5V"/>
+<pinref part="R13" gate="G$1" pin="2"/>
+<wire x1="195.58" y1="127" x2="195.58" y2="124.46" width="0.1524" layer="91"/>
+</segment>
 </net>
 <net name="+12V" class="0">
@@
 </segment>
 </net>
-<net name="N$36" class="0">
-<segment>
-<pinref part="DD20" gate="A" pin="I1"/>
-<wire x1="177.8" y1="109.22" x2="175.26" y2="109.22" width="0.1524" layer="91"/>
-<wire x1="175.26" y1="109.22" x2="175.26" y2="106.68" width="0.1524" layer="91"/>
-<wire x1="175.26" y1="106.68" x2="157.48" y2="106.68" width="0.1524" layer="91"/>
-</segment>
-</net>
 <net name="N$44" class="0">
 <segment>
@@
 <junction x="195.58" y="111.76"/>
 <wire x1="195.58" y1="111.76" x2="198.12" y2="111.76" width="0.1524" layer="91"/>
+<pinref part="R13" gate="G$1" pin="1"/>
+<wire x1="195.58" y1="114.3" x2="195.58" y2="111.76" width="0.1524" layer="91"/>
+</segment>
+</net>
+<net name="STRT" class="0">
+<segment>
+<pinref part="DD20" gate="A" pin="I1"/>
+<wire x1="177.8" y1="109.22" x2="175.26" y2="109.22" width="0.1524" layer="91"/>
+<wire x1="175.26" y1="109.22" x2="175.26" y2="106.68" width="0.1524" layer="91"/>
+<wire x1="175.26" y1="106.68" x2="147.32" y2="106.68" width="0.1524" layer="91"/>
+<label x="149.86" y="106.68" size="1.778" layer="95"/>
+</segment>
+</net>
+<net name="A14" class="0">
+<segment>
+<pinref part="DD11" gate="A" pin="I0"/>
+<wire x1="147.32" y1="116.84" x2="157.48" y2="116.84" width="0.1524" layer="91"/>
+<label x="149.86" y="116.84" size="1.778" layer="95"/>
+</segment>
+</net>
+<net name="A15" class="0">
+<segment>
+<pinref part="DD11" gate="A" pin="I1"/>
+<wire x1="147.32" y1="111.76" x2="157.48" y2="111.76" width="0.1524" layer="91"/>
+<label x="149.86" y="111.76" size="1.778" layer="95"/>
+</segment>
+</net>
+<net name="DD9DD14" class="0">
+<segment>
+<pinref part="DD36" gate="A" pin="1G"/>
+<wire x1="200.66" y1="152.4" x2="195.58" y2="152.4" width="0.1524" layer="91"/>
+<wire x1="195.58" y1="152.4" x2="195.58" y2="142.24" width="0.1524" layer="91"/>
+<pinref part="DD36" gate="A" pin="2C"/>
+<wire x1="195.58" y1="142.24" x2="200.66" y2="142.24" width="0.1524" layer="91"/>
+<wire x1="195.58" y1="142.24" x2="195.58" y2="134.62" width="0.1524" layer="91"/>
+<wire x1="195.58" y1="134.62" x2="220.98" y2="134.62" width="0.1524" layer="91"/>
+<wire x1="220.98" y1="134.62" x2="220.98" y2="111.76" width="0.1524" layer="91"/>
+<pinref part="DD9" gate="C" pin="O"/>
+<wire x1="220.98" y1="111.76" x2="218.44" y2="111.76" width="0.1524" layer="91"/>
+<junction x="195.58" y="142.24"/>
+<wire x1="220.98" y1="111.76" x2="231.14" y2="111.76" width="0.1524" layer="91"/>
+<label x="223.52" y="111.76" size="1.778" layer="95"/>
+<junction x="220.98" y="111.76"/>
+</segment>
+</net>
+<net name="A12" class="0">
+<segment>
+<pinref part="DD36" gate="A" pin="A"/>
+<wire x1="187.96" y1="160.02" x2="200.66" y2="160.02" width="0.1524" layer="91"/>
+<label x="190.5" y="160.02" size="1.778" layer="95"/>
+</segment>
+</net>
+<net name="A11" class="0">
+<segment>
+<pinref part="DD36" gate="A" pin="B"/>
+<wire x1="187.96" y1="157.48" x2="200.66" y2="157.48" width="0.1524" layer="91"/>
+<label x="190.5" y="157.48" size="1.778" layer="95"/>
+</segment>
+</net>
+<net name="A13" class="0">
+<segment>
+<pinref part="DD36" gate="A" pin="2G"/>
+<wire x1="200.66" y1="144.78" x2="198.12" y2="144.78" width="0.1524" layer="91"/>
+<wire x1="198.12" y1="144.78" x2="198.12" y2="149.86" width="0.1524" layer="91"/>
+<pinref part="DD36" gate="A" pin="1C"/>
+<wire x1="198.12" y1="149.86" x2="200.66" y2="149.86" width="0.1524" layer="91"/>
+<wire x1="187.96" y1="149.86" x2="198.12" y2="149.86" width="0.1524" layer="91"/>
+<junction x="198.12" y="149.86"/>
+<label x="190.5" y="149.86" size="1.778" layer="95"/>
 </segment>
 </net>

Commit message: .
Connections:
- net !G19A: now also DD7B.I0
- net !RD: now also DD7B.I2
- net !WE: now also DD7B.O
- net G15: now also DD7B.I1
Changed lines of the file:
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@@
 <instance part="GND41" gate="1" x="187.96" y="132.08" rot="R270"/>
 <instance part="DD14" gate="A" x="264.16" y="101.6"/>
+<instance part="DD7" gate="B" x="203.2" y="81.28"/>
 </instances>
 <busses>
@@
 <wire x1="132.08" y1="213.36" x2="121.92" y2="213.36" width="0.1524" layer="91"/>
 <junction x="132.08" y="218.44"/>
+</segment>
+<segment>
+<pinref part="DD7" gate="B" pin="I1"/>
+<wire x1="180.34" y1="81.28" x2="195.58" y2="81.28" width="0.1524" layer="91"/>
+<label x="182.88" y="81.28" size="1.778" layer="95"/>
 </segment>
 </net>
@@
 <label x="243.84" y="121.92" size="1.778" layer="95"/>
 </segment>
+<segment>
+<pinref part="DD7" gate="B" pin="I2"/>
+<wire x1="180.34" y1="78.74" x2="195.58" y2="78.74" width="0.1524" layer="91"/>
+<label x="182.88" y="78.74" size="1.778" layer="95"/>
+</segment>
 </net>
 <net name="N$69" class="0">
@@
 <label x="243.84" y="99.06" size="1.778" layer="95"/>
 </segment>
-</net>
+<segment>
+<pinref part="DD7" gate="B" pin="I0"/>
+<wire x1="180.34" y1="83.82" x2="195.58" y2="83.82" width="0.1524" layer="91"/>
+<label x="182.88" y="83.82" size="1.778" layer="95"/>
+</segment>
+</net>
+<net name="!WE" class="0">
+<segment>
+<wire x1="180.34" y1="71.12" x2="215.9" y2="71.12" width="0.1524" layer="91"/>
+<wire x1="215.9" y1="71.12" x2="215.9" y2="81.28" width="0.1524" layer="91"/>
+<pinref part="DD7" gate="B" pin="O"/>
+<wire x1="215.9" y1="81.28" x2="210.82" y2="81.28" width="0.1524" layer="91"/>
+<label x="182.88" y="71.12" size="1.778" layer="95"/>
+</segment>
+</net>
