File: b4/SpecialistEE20.brd (EAGLE design)
At the start: 93 parts

Commit message: .
Parts:
- moved DD114 72.1 mm to (38.1, 130.8), turned to 0 degrees
- moved DD112 69.3 mm to (39.4, 144.8), turned to 270 degrees
- moved DD113 53.4 mm to (115.6, 113.0), turned to 0 degrees
- moved DD3011.1 49.5 mm to (97.8, 105.4), turned to 0 degrees
- moved DD30 39.2 mm to (97.8, 113.0), turned to 0 degrees
- moved DD108 38.1 mm to (196.8, 114.3)
- moved DD110 35.6 mm to (163.8, 128.3)
- moved DD3011.2 29.3 mm to (97.8, 120.7), turned to 0 degrees
- moved DD14 24.4 mm to (63.5, 124.5)
- moved DD12 20.8 mm to (62.2, 147.3)
- moved DD33 12.7 mm to (171.4, 111.8)
- moved DD109 12.7 mm to (184.2, 111.8)
- moved DD32 12.7 mm to (158.8, 111.8)
- moved R8 5.39 mm to (189.2, 128.3), turned to 0 degrees
- moved R9 5.24 mm to (176.5, 128.3), turned to 0 degrees
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Routing:
- net VCC: track 81.1 -> 0.00 mm
- net !RD: track 78.8 -> 0.00 mm
- net D7: track 78.5 -> 0.00 mm
- net D6: track 76.1 -> 0.00 mm
- net D5: track 73.8 -> 0.00 mm
- net D4: track 71.7 -> 0.00 mm
- net D3: track 69.7 -> 0.00 mm
- net D2: track 67.9 -> 0.00 mm
- net D1: track 66.3 -> 0.00 mm
- net D0: track 65.0 -> 0.00 mm
- net RES: track 63.9 -> 0.00 mm
- net GND: track 268.8 -> 294.2 mm
