File: b6/SpecialistEE20.brd (EAGLE design)
At the start: 55.9 x 6.6 mm, 104 parts, among them X1 SCART-F

Commit message: .
Parts:
- removed U$1: (no value), simvol-ik:PCB-MAIN
- moved DD19 115.6 mm to (298.4, 21.6)
- moved DD37 115.6 mm to (250.2, 30.5)
- moved DD39 115.6 mm to (273.1, 30.5)
- moved R105 115.6 mm to (208.3, -5.08)
- moved R106 115.6 mm to (209.6, -6.35)
- moved DD38 115.6 mm to (252.7, 64.8)
- moved R9 115.6 mm to (274.3, -14.0)
- moved VD4 115.6 mm to (254.0, -14.0)
- moved VD5 115.6 mm to (259.1, -14.0)
- moved VD6 115.6 mm to (264.2, -14.0)
- moved VD7 115.6 mm to (269.2, -14.0)
- moved R13 101.4 mm to (190.5, 184.2), turned to 180 degrees
- moved R1 98.5 mm to (171.4, 184.2), turned to 180 degrees
- moved Z1 97.0 mm to (177.8, 186.7), turned to 0 degrees
- moved R2 95.5 mm to (180.3, 182.9), turned to 180 degrees
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Routing:
- net N$29: track 33.1 -> 45.8 mm
- net +5V: track 213.5 -> 216.7 mm

Commit message: b
Parts:
- added DD3011.3: (no value), Разъёмы штырьковые 2.54мм:1X20
- moved DD7 15.9 mm to (148.6, 135.9)
- moved DD11 14.9 mm to (148.6, 120.7)
- moved DD6 8.52 mm to (147.3, 151.1)
- moved DD20 6.35 mm to (147.3, 165.1)
- moved DD9 5.24 mm to (147.3, 179.1)
