File: b6/SpecialistEE20.sch (EAGLE design)
At the start: 103 parts, among them X1 SCART-F

Commit message: b
Parts:
- added DD3011.3: (no value), Разъёмы штырьковые 2.54мм:PINHD-1X20
Other:
- note removed: "DD1 использован DD28"
