File: b5/SpecialistEE20.brd (EAGLE design)
At the start: 55.9 x 6.6 mm, 104 parts, among them X1 SCART-F

Commit message: br
Parts:
- removed DD3011.3: (no value), Разъёмы штырьковые 2.54мм:1X20
- removed JP2, JP3: (no value), Разъёмы штырьковые 2.54мм:1X40
- added U$1: (no value), simvol-ik:PCB-MAIN
- moved DD19 115.6 mm to (297.2, -94.0)
- moved DD37 115.6 mm to (248.9, -85.1)
- moved DD39 115.6 mm to (271.8, -85.1)
- moved R105 115.6 mm to (207.0, -120.7)
- moved R106 115.6 mm to (208.3, -121.9)
- moved DD38 115.6 mm to (251.5, -50.8)
- moved R9 115.6 mm to (273.1, -129.5)
- moved VD4 115.6 mm to (252.7, -129.5)
- moved VD5 115.6 mm to (257.8, -129.5)
- moved VD6 115.6 mm to (262.9, -129.5)
- moved VD7 115.6 mm to (268.0, -129.5)
- moved R1 110.5 mm to (204.5, 78.7), turned to 0 degrees
- moved R13 105.5 mm to (185.4, 78.7), turned to 0 degrees
- moved R2 104.0 mm to (195.6, 80.0), turned to 0 degrees
- moved C1 103.5 mm to (200.7, 81.3), turned to 0 degrees
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Routing:
- net MA7: track 337.1 -> 205.8 mm
- net GND: track 281.5 -> 392.8 mm
- net MA6: track 273.8 -> 202.0 mm
- net MA1: track 207.4 -> 162.5 mm
- net MA0: track 211.1 -> 166.4 mm
- net N$50: track 0.00 -> 42.3 mm
- net MA4: track 229.4 -> 191.3 mm
- net N$56: track 0.00 -> 36.9 mm
- net MA2: track 214.5 -> 179.4 mm
- net MA3: track 202.1 -> 169.0 mm
- net N$51: track 0.00 -> 30.0 mm
- net !RD: track 0.00 -> 29.0 mm
- net N$42: track 0.00 -> 28.6 mm
- net D2: track 0.00 -> 22.9 mm
- net D1: track 0.00 -> 22.9 mm
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