File: b5/SpecialistEE20.sch (EAGLE design)
At the start: 104 parts, among them X1 SCART-F

Commit message: br
Parts:
- removed DD3011.3: (no value), Разъёмы штырьковые 2.54мм:PINHD-1X20
- removed JP2, JP3: (no value), Разъёмы штырьковые 2.54мм:PINHD-1X40
Other:
- note added: "DD1 использован DD28"
