File: base/SpecialistEE20.brd (EAGLE design)
At the start: 55.9 x 6.6 mm, 102 parts, among them X1 SCART-F

Commit message: .
Parts:
- moved J1 47.0 mm to (-31.8, 135.9), turned to 0 degrees
- moved 27512 7.62 mm to (110.5, 165.1)
- moved X1 6.48 mm to (57.1, 175.3)
- moved KB 6.35 mm to (100.3, 186.7)
- moved DD113 1.27 mm to (76.2, 115.6)

Commit message: br
Parts:
- removed U$1: (no value), simvol-ik:PCB-MAIN
- added DD3011.3: (no value), Разъёмы штырьковые 2.54мм:1X20
- added JP2, JP3: (no value), Разъёмы штырьковые 2.54мм:1X40
- moved DD19 115.6 mm to (298.4, 21.6)
- moved DD37 115.6 mm to (250.2, 30.5)
- moved DD39 115.6 mm to (273.1, 30.5)
- moved R105 115.6 mm to (208.3, -5.08)
- moved R106 115.6 mm to (209.6, -6.35)
- moved DD38 115.6 mm to (252.7, 64.8)
- moved R9 115.6 mm to (274.3, -14.0)
- moved VD4 115.6 mm to (254.0, -14.0)
- moved VD5 115.6 mm to (259.1, -14.0)
- moved VD6 115.6 mm to (264.2, -14.0)
- moved VD7 115.6 mm to (269.2, -14.0)
- moved R1 110.5 mm to (171.4, 184.2), turned to 180 degrees
- moved R13 105.5 mm to (190.5, 184.2), turned to 180 degrees
- moved R2 104.0 mm to (180.3, 182.9), turned to 180 degrees
- moved C1 103.5 mm to (175.3, 181.6), turned to 180 degrees
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Routing:
- net MA7: track 205.8 -> 337.1 mm
- net GND: track 392.8 -> 281.5 mm
- net MA6: track 202.0 -> 273.8 mm
- net MA1: track 162.5 -> 207.4 mm
- net MA0: track 166.4 -> 211.1 mm
- net N$50: track 42.3 -> 0.00 mm
- net MA4: track 191.3 -> 229.4 mm
- net N$56: track 36.9 -> 0.00 mm
- net MA2: track 179.4 -> 214.5 mm
- net MA3: track 169.0 -> 202.1 mm
- net N$51: track 30.0 -> 0.00 mm
- net !RD: track 29.0 -> 0.00 mm
- net N$42: track 28.6 -> 0.00 mm
- net D2: track 22.9 -> 0.00 mm
- net D1: track 22.9 -> 0.00 mm
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
Commit message: .
Parts:
- added R11B: 2k, rcl:M1206
- renumbered DD113 to DD213, DD114 to DD214
Connections:
- removed net A'11: DD16.11
- removed net A'12: DD17.5
- removed net A'13: DD17.11
- removed net A'14: DD18.10
- removed net A'15: DD18.11
- new net N$67: DD18.13, R11B.1
- net +5V: now also R11B.2
- net A11: now also DD16.11
- net A12: now also DD17.5
- net A13: now also DD17.11
- net A14: now also DD18.10
- net A15: now also DD18.11
- net N$31: no longer DD18.13

Commit message: c
Parts:
- moved DD34 1.27 mm to (88.9, 90.2)
Connections:
- removed net N$41: DD15.14, DD16.14, DD17.14, DD18.14
- removed net N$49: DD32.8, DD33.8, R23.1
- net !RAS: now also DD15.14, DD16.14, DD17.14, DD18.14
- net +5V: now also DD112.26, DD30.26
- net R2: now also DD32.8, DD33.8, R23.1
- net VCC: no longer DD112.26, DD30.26
Routing:
- net +5V: track 216.7 -> 211.1 mm

Commit message: .
Routing:
- net +5V: track 211.1 -> 190.8 mm
Changed lines of the file:
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@@
 <contactref element="RD1" pad="2"/>
 <contactref element="RD2" pad="1"/>
-<contactref element="DD21" pad="8"/>
-<contactref element="DD28" pad="8"/>
-<contactref element="DD27" pad="8"/>
-<contactref element="DD26" pad="8"/>
-<contactref element="DD25" pad="8"/>
-<contactref element="DD24" pad="8"/>
-<contactref element="DD23" pad="8"/>
-<contactref element="DD22" pad="8"/>
 <contactref element="DD102" pad="8"/>
 <contactref element="DD103" pad="8"/>
@@
 <wire x1="49.53" y1="1.27" x2="38.1" y2="1.27" width="1.9304" layer="16"/>
 <wire x1="38.1" y1="1.27" x2="25.4" y2="1.27" width="1.9304" layer="16"/>
-<wire x1="63.5" y1="3.81" x2="63.5" y2="1.27" width="1.4224" layer="16"/>
-<wire x1="76.2" y1="3.81" x2="76.2" y2="1.27" width="1.4224" layer="16"/>
-<wire x1="88.9" y1="3.81" x2="88.9" y2="1.27" width="1.4224" layer="16"/>
-<wire x1="101.6" y1="3.81" x2="101.6" y2="1.27" width="1.4224" layer="16"/>
-<wire x1="114.3" y1="3.81" x2="114.3" y2="1.27" width="1.4224" layer="16"/>
-<wire x1="127" y1="3.81" x2="127" y2="1.27" width="1.4224" layer="16"/>
-<wire x1="139.7" y1="3.81" x2="139.7" y2="1.27" width="1.4224" layer="16"/>
-<wire x1="152.4" y1="1.27" x2="152.4" y2="3.81" width="1.4224" layer="16"/>
 <contactref element="R106" pad="2"/>
 <contactref element="R105" pad="2"/>
@@
 <contactref element="DD107" pad="14"/>
 <contactref element="DD112" pad="26"/>
+<contactref element="DD21" pad="8"/>
+<contactref element="DD22" pad="8"/>
+<contactref element="DD23" pad="8"/>
+<contactref element="DD24" pad="8"/>
+<contactref element="DD28" pad="8"/>
+<contactref element="DD27" pad="8"/>
+<contactref element="DD26" pad="8"/>
+<contactref element="DD25" pad="8"/>
 <wire x1="125.6" y1="107.95" x2="124.33" y2="115.57" width="0" layer="19" extent="1-16"/>
 <wire x1="116.84" y1="107.95" x2="125.6" y2="107.95" width="0" layer="19" extent="16-16"/>
@@
 <wire x1="208.6" y1="-6.35" x2="207.33" y2="-5.08" width="0" layer="19" extent="16-16"/>
 <wire x1="152.4" y1="1.27" x2="207.33" y2="-5.08" width="0" layer="19" extent="16-16"/>
+<wire x1="152.4" y1="3.81" x2="152.4" y2="1.27" width="0" layer="19" extent="16-16"/>
+<wire x1="139.7" y1="3.81" x2="139.7" y2="1.27" width="0" layer="19" extent="16-16"/>
+<wire x1="127" y1="3.81" x2="127" y2="1.27" width="0" layer="19" extent="16-16"/>
+<wire x1="114.3" y1="3.81" x2="114.3" y2="1.27" width="0" layer="19" extent="16-16"/>
+<wire x1="101.6" y1="3.81" x2="101.6" y2="1.27" width="0" layer="19" extent="16-16"/>
+<wire x1="88.9" y1="3.81" x2="88.9" y2="1.27" width="0" layer="19" extent="16-16"/>
+<wire x1="76.2" y1="3.81" x2="76.2" y2="1.27" width="0" layer="19" extent="16-16"/>
+<wire x1="63.5" y1="3.81" x2="63.5" y2="1.27" width="0" layer="19" extent="16-16"/>
 <wire x1="274.32" y1="-15.37" x2="208.6" y2="-6.35" width="0" layer="19" extent="16-16"/>
 <wire x1="307.34" y1="17.78" x2="274.32" y2="-15.37" width="0" layer="19" extent="16-16"/>

Commit message: ..
Parts:
- added DDX12A: (no value), Разъёмы штырьковые 2.54мм:1X20
- added DDX12B: (no value), Разъёмы штырьковые 2.54мм:1X04
- added DDX12C: (no value), Разъёмы штырьковые 2.54мм:1X06
- added ISP_KB, ISP_SD: (no value), con-lstb:MA03-2
- moved KB 63.5 mm to (36.8, 186.7)
- moved J1 54.8 mm to (61.0, 165.1)
- moved X1 49.5 mm to (106.7, 176.5)
- moved DD45 29.2 mm to (203.2, 105.4), turned to 0 degrees
- moved DD14 28.8 mm to (101.6, 161.3)
- moved DD36 14.0 mm to (101.6, 147.3)
- moved DD20 13.0 mm to (160.0, 162.6)
- moved DD9 10.2 mm to (157.5, 179.1)
- moved 27512 9.25 mm to (102.9, 125.7)
- moved DD12 4.58 mm to (127.0, 163.8)
Connections:
- net N$35 renamed PS2C
- net N$39 renamed PS2D
- removed net K26: DD30.11
- net !RESIN: now also ISP_KB.5, ISP_SD.5
- net !U6: now also DD36.5
- net +5V: now also ISP_KB.2, ISP_SD.2
- net B: now also DD30.13
- net G: now also DD30.11
- net GND: now also ISP_KB.6, ISP_SD.6
- net K1: now also ISP_KB.4
- net K5: now also ISP_KB.1
- net K6: now also ISP_KB.3
- net MISO: now also ISP_SD.1
- net MOSI: now also ISP_SD.4
- net R: now also DD30.10
- net SCK: now also ISP_SD.3
- net SND: now also DD30.12

Commit message: .
Parts:
- removed DD3011.3: (no value), Разъёмы штырьковые 2.54мм:1X20
- moved DDX12B 245.4 mm to (58.4, 156.2), turned to 270 degrees
- moved DDX12C 205.4 mm to (58.4, 118.1), turned to 270 degrees
- moved DDX12A 191.8 mm to (35.6, 135.9), turned to 270 degrees
- moved R11B 52.9 mm to (-30.5, 16.5)
- moved ISP_KB 38.4 mm to (80.0, 165.1)
- moved ISP_SD 24.4 mm to (40.6, 165.1)
- moved KB 24.2 mm to (61.0, 188.0)
- moved DD108 22.9 mm to (26.7, 90.2)
- moved DD110 22.9 mm to (26.7, 114.3)
- moved R102 15.5 mm to (22.9, 157.5)
- moved R101 13.7 mm to (22.9, 163.8)
- moved J1 12.8 mm to (59.7, 177.8)
- moved DD14 11.5 mm to (113.0, 160.0)
- moved R103 10.8 mm to (26.7, 170.2)
- moved DD28 10.5 mm to (153.7, 22.9)
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Connections:
- net !RD: now also DDX12A.5
- net !U6: now also DDX12A.6
- net A0: now also DDX12A.9
- net A1: now also DDX12A.8
- net GND: now also DDX12A.7
- net P1: now also DDX12A.4
- net P10: now also DDX12A.19
- net P11: now also DDX12A.20
- net P12: now also DDX12C.6
- net P13: now also DDX12C.5
- net P14: now also DDX12C.4
- net P15: now also DDX12C.3
- net P16: now also DDX12C.2
- net P17: now also DDX12A.14
- net P18: now also DDX12A.15
- net P19: now also DDX12A.16
- net P2: now also DDX12A.3
- net P20: now also DDX12A.17
- net P21: now also DDX12A.13
- net P22: now also DDX12A.12
- net P23: now also DDX12A.11
- net P24: now also DDX12A.10
- net P3: now also DDX12A.2
- net P4: now also DDX12A.1
- net P5: now also DDX12B.1
- net P6: now also DDX12B.2
- net P7: now also DDX12B.3
- net P8: now also DDX12B.4
- net P9: now also DDX12A.18
Routing:
- net VID: track 353.1 -> 289.6 mm
- net D5: track 0.00 -> 32.8 mm
- net D4: track 0.00 -> 32.8 mm
- net D3: track 0.00 -> 32.8 mm
- net D1: track 0.00 -> 32.8 mm
- net D0: track 0.00 -> 32.8 mm
- net A0: track 0.00 -> 32.8 mm
- net D7: track 0.00 -> 32.8 mm
- net D6: track 0.00 -> 32.8 mm
- net A1: track 0.00 -> 32.8 mm
- net !RD: track 0.00 -> 32.8 mm
- net D2: track 0.00 -> 29.0 mm
- net MA4: track 229.4 -> 219.0 mm
- net MA2: track 214.5 -> 204.1 mm
- net MA5: track 209.4 -> 199.0 mm
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
Commit message: .
Parts:
- moved J1 12.7 mm to (59.7, 165.1)
- moved KB 4.58 mm to (58.4, 184.2)
Changed lines of the file:
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@@
 <board>
 <plain>
-<dimension x1="191.77" y1="199.39" x2="24.13" y2="208.28" x3="107.95" y3="54.61" textsize="1.778" layer="21" dtype="horizontal"/>
-<dimension x1="15.24" y1="73.66" x2="19.05" y2="189.23" x3="243.84" y3="131.445" textsize="1.778" layer="21" dtype="vertical"/>
+<dimension x1="190.5" y1="207.01" x2="19.05" y2="199.39" x3="104.775" y3="54.61" textsize="1.778" layer="21" dtype="horizontal"/>
+<dimension x1="15.24" y1="73.66" x2="12.7" y2="185.42" x3="228.6" y3="129.54" textsize="1.778" layer="21" dtype="vertical"/>
 <text x="248.92" y="93.98" size="6.4516" layer="22" rot="R180">21x13</text>
 <text x="228.6" y="121.92" size="6.4516" layer="22">220х135 вост экс нов</text>
@@
 <element name="DD3011.1" library="Разъёмы штырьковые 2.54мм" package="1X20" value="" x="63.5" y="135.89" rot="R270"/>
 <element name="DD3011.2" library="Разъёмы штырьковые 2.54мм" package="1X20" value="" x="86.36" y="135.89" rot="R270"/>
-<element name="KB" library="Speccy" package="MINI-DIN6" value="MINI-DIN6" x="60.96" y="187.96"/>
+<element name="KB" library="Speccy" package="MINI-DIN6" value="MINI-DIN6" x="58.42" y="184.15"/>
 <element name="DD45" library="74xx-eu" package="DIL14" value="К555ИЕ19" x="203.2" y="105.41"/>
 <element name="R105" library="rcl" package="M0805" value="4k7" x="208.28" y="-5.08" rot="MR0"/>
@@
 <attribute name="OC_FARNELL" value="unknown" x="106.68" y="176.53" size="1.778" layer="27" rot="R180" display="off"/>
 </element>
-<element name="J1" library="Speccy" package="SDCMF-10915W010" value="" x="59.69" y="177.8" rot="R180"/>
+<element name="J1" library="Speccy" package="SDCMF-10915W010" value="" x="59.69" y="165.1" rot="R180"/>
 <element name="U$2" library="ESR_NM8032" package="SWITCH9X4" value="SWITCH9X4" x="-12.7" y="152.4"/>
 <element name="R13" library="rcl" package="M1206" value="2k" x="190.5" y="184.15" rot="R180"/>
@@
 <wire x1="102.87" y1="152.4" x2="105.41" y2="163.83" width="0" layer="19" extent="1-1"/>
 <wire x1="82.55" y1="166.37" x2="105.41" y2="163.83" width="0" layer="19" extent="1-1"/>
-<wire x1="73.136125" y1="166.37" x2="82.55" y2="166.37" width="0" layer="19" extent="1-1"/>
-<wire x1="72.898" y1="180.34" x2="73.136125" y2="166.37" width="0" layer="19" extent="1-1"/>
-<wire x1="64.36" y1="179.46" x2="72.898" y2="180.34" width="0" layer="19" extent="1-1"/>
-<wire x1="45.72" y1="180.34" x2="64.36" y2="179.46" width="0" layer="19" extent="1-1"/>
-<wire x1="47.259875" y1="166.37" x2="45.72" y2="180.34" width="0" layer="19" extent="1-1"/>
-<wire x1="43.18" y1="166.37" x2="47.259875" y2="166.37" width="0" layer="19" extent="1-1"/>
+<wire x1="73.136125" y1="153.67" x2="82.55" y2="166.37" width="0" layer="19" extent="1-1"/>
+<wire x1="72.898" y1="167.64" x2="73.136125" y2="153.67" width="0" layer="19" extent="1-1"/>
+<wire x1="61.82" y1="175.65" x2="72.898" y2="167.64" width="0" layer="19" extent="1-1"/>
+<wire x1="45.72" y1="167.64" x2="61.82" y2="175.65" width="0" layer="19" extent="1-1"/>
+<wire x1="47.259875" y1="153.67" x2="45.72" y2="167.64" width="0" layer="19" extent="1-1"/>
+<wire x1="43.18" y1="166.37" x2="47.259875" y2="153.67" width="0" layer="19" extent="1-1"/>
 <wire x1="24.13" y1="170.18" x2="43.18" y2="166.37" width="0" layer="19" extent="1-1"/>
 <wire x1="20.32" y1="163.83" x2="24.13" y2="170.18" width="0" layer="19" extent="1-1"/>
@@
 <contactref element="ISP_SD" pad="2"/>
 <contactref element="ISP_KB" pad="2"/>
-<wire x1="57.56" y1="179.46" x2="77.47" y2="166.37" width="0" layer="19" extent="1-1"/>
-<wire x1="38.1" y1="166.37" x2="57.56" y2="179.46" width="0" layer="19" extent="1-1"/>
+<wire x1="55.02" y1="175.65" x2="77.47" y2="166.37" width="0" layer="19" extent="1-1"/>
+<wire x1="38.1" y1="166.37" x2="55.02" y2="175.65" width="0" layer="19" extent="1-1"/>
 <wire x1="48.99" y1="136.3726" x2="38.1" y2="166.37" width="0" layer="19" extent="1-1"/>
 <wire x1="48.19" y1="127.7874" x2="48.99" y2="136.3726" width="0" layer="19" extent="1-1"/>
@@
 <contactref element="DD213" pad="1"/>
 <contactref element="R106" pad="1"/>
-<wire x1="79" y1="118.5926" x2="62.26" y2="179.46" width="0" layer="19" extent="1-1"/>
+<wire x1="79" y1="118.5926" x2="59.72" y2="175.65" width="0" layer="19" extent="1-1"/>
 <wire x1="210.5" y1="-6.35" x2="79" y2="118.5926" width="0" layer="19" extent="1-16"/>
 </signal>
@@
 <contactref element="KB" pad="1"/>
 <contactref element="R105" pad="1"/>
-<wire x1="71.9074" y1="116.3" x2="59.66" y2="179.46" width="0" layer="19" extent="1-1"/>
+<wire x1="71.9074" y1="116.3" x2="57.12" y2="175.65" width="0" layer="19" extent="1-1"/>
 <wire x1="209.23" y1="-5.08" x2="71.9074" y2="116.3" width="0" layer="19" extent="1-16"/>
 </signal>
