File: base/SpecialistEE20.brd (EAGLE design)
At the start: 55.9 x 6.6 mm, 109 parts, among them X1 SCART-F

Commit message: s
Parts:
- moved DD110 54.7 mm to (29.2, 168.9), turned to 0 degrees
- moved DD107 53.4 mm to (-5.08, 125.7)
- moved R102 26.2 mm to (29.2, 182.9), turned to 180 degrees
- moved R101 17.1 mm to (34.3, 176.5), turned to 180 degrees
- moved DD14 16.7 mm to (96.5, 162.6)
- moved R103 15.3 mm to (40.6, 176.5), turned to 180 degrees
- moved DD36 13.0 mm to (99.1, 146.1)
- moved 27512 10.2 mm to (102.9, 123.2)
- moved DD29 7.62 mm to (127.0, 132.1)
- moved X1 2.54 mm to (106.7, 174.0)
- turned DD109 to 270 degrees
Connections:
- net !G19A renamed !G19T
- net N$33 renamed K21
- removed net N$57: DD14.6, DD14.9
- removed net RES80: DD12.6, DD29.12
- new net !RES: DD12.5, DD14.4
- net B: now also DD14.10
- net GND: now also X1.13, X1.14, X1.17, X1.18, X1.21, X1.4, X1.5, X1.9
- net RES: now also DD12.6, DD29.12
- net STRT: now also DD14.6, DD14.9
Routing:
- net GND: track 281.5 -> 367.8 mm
- net R2: track 0.00 -> 59.0 mm
- net MA7: track 327.4 -> 276.6 mm
- net VD7: track 0.00 -> 38.4 mm
- net VD5: track 0.00 -> 29.3 mm
- net Q3: track 0.00 -> 27.5 mm
- net CLK: track 0.00 -> 27.5 mm
- net VD6: track 0.00 -> 22.4 mm
- net VD1: track 0.00 -> 18.1 mm
- net N$43: track 0.00 -> 17.3 mm
- net N$46: track 0.00 -> 13.8 mm
- net N$45: track 0.00 -> 13.8 mm
- net VD3: track 0.00 -> 11.2 mm
- net VD2: track 0.00 -> 11.2 mm

Commit message: s
Parts:
- added R7'': 4k7, rcl:M0805
- S1: value SWITCH9X4 -> TapeOn
- moved DD14 4.58 mm to (99.1, 158.8)
- moved ISP_KB 1.80 mm to (78.7, 166.4), turned to 90 degrees
- moved ISP_SD 1.80 mm to (41.9, 166.4), turned to 270 degrees
- moved DD36 1.80 mm to (100.3, 147.3)
- renumbered U$2 to S1
Connections:
- new net N$35: S1.11, S1.21
- net +5V: now also R7''.2
- net GND: now also S1.12, S1.22
- net TON: now also R7''.1, S1.10, S1.20
