File: base/SpecialistEE20.sch (EAGLE design)
At the start: 101 parts, among them X1 SCART-F

Commit message: br
Parts:
- added DD3011.3: (no value), Разъёмы штырьковые 2.54мм:PINHD-1X20
- added JP2, JP3: (no value), Разъёмы штырьковые 2.54мм:PINHD-1X40
Other:
- note removed: "DD1 использован DD28"

Commit message: .
Parts:
- removed DD113, DD114: MEGA8-AI, atmel:MEGA8-AI
- added DD213, DD214: MEGA8-AI, atmel:MEGA8-AI
- added R11B: 2k, rcl:R-EU_M1206
Connections:
- removed net A'11: DD16A.2C1
- removed net A'12: DD17A.1C1
- removed net A'13: DD17A.2C1
- removed net A'14: DD18A.2C0
- removed net A'15: DD18A.2C1
- new net N$67: DD18A.2C3, R11B.1
- net !R: now also DD214.PC1(ADC1); no longer DD114.PC1(ADC1)
- net !RESIN: now also DD213.PC6(/RESET), DD214.PC6(/RESET); no longer DD113.PC6(/RESET), DD114.PC6(/RESET)
- net +5V: now also DD213.AVCC, DD213.VCC@1, DD213.VCC@2, DD214.AVCC, DD214.VCC@1, DD214.VCC@2, R11B.2; no longer DD113.AVCC, DD113.VCC@1, DD113.VCC@2, DD114.AVCC, DD114.VCC@1, DD114.VCC@2
- net A11: now also DD16A.2C1
- net A12: now also DD17A.1C1
- net A13: now also DD17A.2C1
- net A14: now also DD18A.2C0
- net A15: now also DD18A.2C1
- net CS: now also DD214.PB2(SS/OC1B); no longer DD114.PB2(SS/OC1B)
- net GND: now also DD213.GND, DD213.GND@1, DD213.GND@2, DD214.GND, DD214.GND@1, DD214.GND@2; no longer DD113.GND, DD113.GND@1, DD113.GND@2, DD114.GND, DD114.GND@1, DD114.GND@2
- net K1: now also DD213.PB3(MOSI/OC2); no longer DD113.PB3(MOSI/OC2)
- net K10: now also DD213.PC4(ADC4/SDA); no longer DD113.PC4(ADC4/SDA)
- net K11: now also DD213.PC3(ADC3); no longer DD113.PC3(ADC3)
- net K12: now also DD213.PC2(ADC2); no longer DD113.PC2(ADC2)
- net K13: now also DD213.PD0(RXD); no longer DD113.PD0(RXD)
- net K14: now also DD213.PD1(TXD); no longer DD113.PD1(TXD)
- net K15: now also DD213.PD4(XCK/T0); no longer DD113.PD4(XCK/T0)
- net K16: now also DD213.PD5(T1); no longer DD113.PD5(T1)
- net K17: now also DD213.PC1(ADC1); no longer DD113.PC1(ADC1)
- net K18: now also DD213.PC0(ADC0); no longer DD113.PC0(ADC0)
- net K19: now also DD213.PD7(AIN1); no longer DD113.PD7(AIN1)
- net K2: now also DD213.PB2(SS/OC1B); no longer DD113.PB2(SS/OC1B)
- net K3: now also DD213.PB1(OC1A); no longer DD113.PB1(OC1A)
- net K4: now also DD213.PB0(ICP); no longer DD113.PB0(ICP)
- net K5: now also DD213.PB4(MISO); no longer DD113.PB4(MISO)
- net K6: now also DD213.PB5(SCK), DD213.PB6(XTAL1/TOSC1); no longer DD113.PB5(SCK), DD113.PB6(XTAL1/TOSC1)
- net K8: now also DD213.PB7(XTAL2/TOSC2); no longer DD113.PB7(XTAL2/TOSC2)
- net K9: now also DD213.PC5(ADC5/SCL); no longer DD113.PC5(ADC5/SCL)
- net LED: now also DD214.PB0(ICP); no longer DD114.PB0(ICP)
- net MISO: now also DD214.PB4(MISO); no longer DD114.PB4(MISO)
- net MOSI: now also DD214.PB3(MOSI/OC2); no longer DD114.PB3(MOSI/OC2)
- net N$31: no longer DD18A.2C3
- net N$35: now also DD213.PD3(INT1); no longer DD113.PD3(INT1)
- net N$39: now also DD213.PD6(AIN0); no longer DD113.PD6(AIN0)
- net P16: now also DD214.PC0(ADC0); no longer DD114.PC0(ADC0)
- net P17: now also DD214.PD0(RXD); no longer DD114.PD0(RXD)
- net P18: now also DD214.PD1(TXD); no longer DD114.PD1(TXD)
- net P19: now also DD214.PD2(INT0); no longer DD114.PD2(INT0)
- net P20: now also DD214.PD3(INT1); no longer DD114.PD3(INT1)
- net P21: now also DD214.PD4(XCK/T0); no longer DD114.PD4(XCK/T0)
- net P22: now also DD214.PD5(T1); no longer DD114.PD5(T1)
- net P23: now also DD214.PD6(AIN0); no longer DD114.PD6(AIN0)
- net P24: now also DD214.PD7(AIN1); no longer DD114.PD7(AIN1)
- net SCK: now also DD214.PB5(SCK); no longer DD114.PB5(SCK)
- net TON: now also DD214.PC2(ADC2); no longer DD114.PC2(ADC2)
- net U7: now also DD213.PD2(INT0); no longer DD113.PD2(INT0)
Other:
- note added: "RAM"

Commit message: c
Connections:
- removed net N$41: DD15A.A, DD16A.A, DD17A.A, DD18A.A
- removed net N$49: DD32A.CK2, DD33A.CK2, R23.1
- net !RAS: now also DD15A.A, DD16A.A, DD17A.A, DD18A.A
- net +5V: now also DD112P.VCC, DD30P.VCC
- net GND: now also DD112P.GND, DD30P.GND
- net R2: now also DD32A.CK2, DD33A.CK2, R23.1
Other:
- moved on the sheet: C10, C11, C3, C4, C4', C6, DD10, DD107A, DD107B, DD107P, DD108, DD108P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

Commit message: .
Other:
- moved on the sheet: DD14A, DD14D, DD21, DD22, DD23, DD24, DD25, DD26, DD27, DD28, DD34

Commit message: ..
Parts:
- added DDX12A: (no value), Разъёмы штырьковые 2.54мм:PINHD-1X20
- added DDX12B: (no value), Разъёмы штырьковые 2.54мм:PINHD-1X4
- added DDX12C: (no value), Разъёмы штырьковые 2.54мм:PINHD-1X6
- added ISP_KB, ISP_SD: (no value), con-lstb:MA03-2
Connections:
- net N$35 renamed PS2C
- net N$39 renamed PS2D
- removed net K26: DD30A.PC6
- net !RESIN: now also ISP_KB.5, ISP_SD.5
- net !U6: now also DD36A.1Y2
- net +5V: now also ISP_KB.2, ISP_SD.2
- net B: now also DD30A.PC4
- net G: now also DD30A.PC6
- net GND: now also ISP_KB.6, ISP_SD.6
- net K1: now also ISP_KB.4
- net K5: now also ISP_KB.1
- net K6: now also ISP_KB.3
- net MISO: now also ISP_SD.1
- net MOSI: now also ISP_SD.4
- net R: now also DD30A.PC7
- net SCK: now also ISP_SD.3
- net SND: now also DD30A.PC5

Commit message: .
Parts:
- removed DD3011.3: (no value), Разъёмы штырьковые 2.54мм:PINHD-1X20
Connections:
- net !RD: now also DDX12A.5
- net !U6: now also DDX12A.6
- net A0: now also DDX12A.9
- net A1: now also DDX12A.8
- net GND: now also DDX12A.7
- net P1: now also DDX12A.4
- net P10: now also DDX12A.19
- net P11: now also DDX12A.20
- net P12: now also DDX12C.6
- net P13: now also DDX12C.5
- net P14: now also DDX12C.4
- net P15: now also DDX12C.3
- net P16: now also DDX12C.2
- net P17: now also DDX12A.14
- net P18: now also DDX12A.15
- net P19: now also DDX12A.16
- net P2: now also DDX12A.3
- net P20: now also DDX12A.17
- net P21: now also DDX12A.13
- net P22: now also DDX12A.12
- net P23: now also DDX12A.11
- net P24: now also DDX12A.10
- net P3: now also DDX12A.2
- net P4: now also DDX12A.1
- net P5: now also DDX12B.1
- net P6: now also DDX12B.2
- net P7: now also DDX12B.3
- net P8: now also DDX12B.4
- net P9: now also DDX12A.18
Other:
- note added: "PS/2 KB & SD Card"
- note added: "Video"
- moved on the sheet: 27512, DD11A, DD20A, DD36, DD37, DD38, DD39, DD45A, DD45B, DD9C, DDX12B, DDX12C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

Commit message: s
Connections:
- net !G19A renamed !G19T
- net N$33 renamed K21
- removed net N$57: DD14B.O, DD14C.I0
- removed net RES80: DD12A.!Q, DD29.RESET
- new net !RES: DD12A.Q, DD14B.I0
- net B: now also DD14C.I1
- net GND: now also X1.13, X1.14, X1.17, X1.18, X1.21, X1.4, X1.5, X1.9
- net RES: now also DD12A.!Q, DD29.RESET
- net STRT: now also DD14B.O, DD14C.I0
