File: base/SpecialistEE20.sch (EAGLE design)
At the start: 109 parts, among them X1 SCART-F

Commit message: s
Parts:
- removed U$2: SWITCH9X4, ESR_NM8032:SWITCH9X4
- added R7'': 4k7, rcl:R-EU_M0805
- added S1: TapeOn, ESR_NM8032:SWITCH9X4
Connections:
- new net N$35: S1A.O, S1B.O
- net +5V: now also R7''.2
- net GND: now also S1A.S, S1B.S
- net TON: now also R7''.1, S1A.P, S1B.P
Other:
- moved on the sheet: DD112, DD29, J1, R14
