File: eagle6.4/Specialist.brd (EAGLE design)
At the start: 55.9 x 6.6 mm, 110 parts, among them X1 SCART-F

Commit message: .
Connections:
- new net !OE!DD37: DD36.9, DD37.20
- new net !OE!DD38: DD36.10, DD38.20
- new net N$33: DD37.18, DD38.18, DD39.22
- new net ROMDD39: DD39.20, R9.1, VD4.A, VD5.A, VD6.A, VD7.A
- net +5V: now also DD37.21, DD38.21, DD39.1, DD39.27
- net GND: now also 27512.1, 27512.26, 27512.27
- net N$18: now also 27512.2; no longer R9.1, VD4.A, VD5.A, VD6.A, VD7.A

Commit message: xm
Parts:
- removed JP3: (no value), Разъёмы штырьковые 2.54мм:1X40
- added JP4: (no value), Разъёмы штырьковые 2.54мм:2X30
- added JP8: (no value), Разъёмы штырьковые 2.54мм:2X03
- added U$1: (no value), Specialist:RAM3+8
- added XCIRGB: (no value), Разъёмы штырьковые 2.54мм:1X07
- added XR1, XR2, XRB, XRB1, XRB3: (no value), Разъёмы штырьковые 2.54мм:2X01
- added XRG, XRG1: (no value), Разъёмы штырьковые 2.54мм:2X02
- JP2: device Разъёмы штырьковые 2.54мм:1X40 -> Разъёмы штырьковые 2.54мм:2X30
- moved JP2 44.1 mm to (55.9, 40.6)
- moved LED1 33.9 mm to (44.5, 208.3)
- moved R107 27.7 mm to (38.1, 199.4)
Connections:
- removed net B0: DD104.14, DD108.7
- removed net G0: DD103.14, DD108.4
- removed net R0: DD102.14, DD108.3
- new net BO: DD104.14, DD108.7, XRB.1, XRB.2, XRB1.1, XRB1.2
- new net GO: DD103.14, DD108.4, XRG.3, XRG.4, XRG1.3, XRG1.4
- new net RO: DD102.14, DD108.3, XRG.1, XRG.2, XRG1.1, XRG1.2
- net B: now also XCIRGB.6, XCIRGB.7, XR1.1, XR1.2
- net G: now also XCIRGB.4, XCIRGB.5, XRB3.1, XRB3.2
- net R: now also XCIRGB.1, XCIRGB.2, XR2.1, XR2.2
Routing:
- net CRG: track 0.00 -> 51.9 mm
- net RO: track 0.00 -> 45.3 mm
- net GO: track 0.00 -> 32.6 mm
- net BO: track 0.00 -> 23.9 mm
- net R0: track 19.1 -> 0.00 mm
- net B: track 3.81 -> 20.6 mm
- net G: track 3.81 -> 20.1 mm
- net GND: track 367.8 -> 378.2 mm
- net B0: track 9.94 -> 0.00 mm
- net R: track 3.81 -> 13.2 mm
- net G0: track 4.34 -> 0.00 mm

Commit message: .
Routing:
- net D2: track 29.0 -> 90.0 mm
- net D7: track 32.8 -> 76.0 mm
- net MD7: track 8.03 -> 40.9 mm
- net GND: track 378.2 -> 408.7 mm
- net MD2: track 8.03 -> 38.1 mm
- net MD0: track 8.03 -> 33.8 mm
- net MD6: track 8.03 -> 33.7 mm
- net MD3: track 8.03 -> 33.0 mm
- net MD5: track 8.03 -> 30.5 mm
- net +5V: track 190.8 -> 210.8 mm
- net MD4: track 8.03 -> 23.6 mm

Commit message: .
Parts:
- added U$2: (no value), nanoitx:NANOITXPCB
- added U$3: (no value), Specialist:RAM3+8
- moved JP1 83.7 mm to (205.7, 146.1)
- moved LED1 63.2 mm to (20.3, 149.9)
- moved R107 43.8 mm to (25.4, 157.5)
- moved S1 42.6 mm to (29.2, 144.8)
- moved R7'' 38.2 mm to (8.89, 67.3)
- moved R11B 37.0 mm to (5.08, 26.7)
- moved DD107 29.2 mm to (24.1, 124.5), turned to 90 degrees
- moved C4 1.80 mm to (135.9, 54.6)
Routing:
- net MA7: track 276.6 -> 201.3 mm
- net MA6: track 263.6 -> 195.1 mm
- net MA4: track 219.0 -> 192.2 mm
- net MA2: track 204.1 -> 197.4 mm
- net MA5: track 199.0 -> 193.9 mm
- net MA0: track 201.4 -> 197.8 mm
- net MA1: track 197.7 -> 196.1 mm
