File: eagle6.4/Specialist.sch (EAGLE design)
At the start: 110 parts, among them X1 SCART-F

Commit message: .
Connections:
- new net !OE!DD37: DD36A.2Y0, DD37A.!OE
- new net !OE!DD38: DD36A.2Y1, DD38A.!OE
- new net N$33: DD37A.!CE, DD38A.!CE, DD39A.!OE
- new net ROMDD39: DD39A.!CE, R9.1, VD4.A, VD5.A, VD6.A, VD7.A
- net +5V: now also DD37A.VPP, DD38A.VPP, DD39A.!PGM, DD39A.VPP
- net GND: now also 27512A.A13, 27512A.A14, 27512A.A15
- net N$18: now also 27512A.A12; no longer R9.1, VD4.A, VD5.A, VD6.A, VD7.A
Other:
- note added: "dd37 dd38 dd39 09 oedd37 1 0 1 10 oedd38 1 1 0 d romdd39 1 1 1"
- note added: "test norm sd a13 0 0 1 a14 0 0 0 a15 0 0 0"
- moved on the sheet: 27512, DD11A, DD20A, DD36, DD37, DD38, DD39, DD9C, R13, R9, VD4, VD5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

Commit message: xm
Parts:
- removed JP3: (no value), Разъёмы штырьковые 2.54мм:PINHD-1X40
- added JP4: (no value), Разъёмы штырьковые 2.54мм:PINHD-2X30
- added JP8: (no value), Разъёмы штырьковые 2.54мм:PINHD-2X3
- added XCIRGB: (no value), Разъёмы штырьковые 2.54мм:PINHD-1X7
- added XR1, XR2, XRB, XRB1, XRB3: (no value), Разъёмы штырьковые 2.54мм:PINHD-1X2
- added XRG, XRG1: (no value), Разъёмы штырьковые 2.54мм:PINHD-2X2
- JP2: device Разъёмы штырьковые 2.54мм:PINHD-1X40 -> Разъёмы штырьковые 2.54мм:PINHD-2X30
Connections:
- removed net B0: DD104.DO, DD108A.3D
- removed net G0: DD103.DO, DD108A.2D
- removed net R0: DD102.DO, DD108A.1D
- new net BO: DD104.DO, DD108A.3D, XRB.1, XRB.2, XRB1.1, XRB1.2
- new net GO: DD103.DO, DD108A.2D, XRG.3, XRG.4, XRG1.3, XRG1.4
- new net RO: DD102.DO, DD108A.1D, XRG.1, XRG.2, XRG1.1, XRG1.2
- net B: now also XCIRGB.6, XCIRGB.7, XR1.1, XR1.2
- net G: now also XCIRGB.4, XCIRGB.5, XRB3.1, XRB3.2
- net R: now also XCIRGB.1, XCIRGB.2, XR2.1, XR2.2

Commit message: .
Other:
- note added: "Панельки DIP14 15 DIP16 19 DIP20 3 DIP24 (2) DIP28 1 (2) DIP40 3"
Changed lines of the file:
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@@
 DD113,DD114 ATMega8
 DA1 КР544УД2</text>
+<text x="162.56" y="109.22" size="1.778" layer="98" rot="MR180">Панельки
+DIP14 15
+DIP16 19
+DIP20 3
+DIP24 (2)
+DIP28 1 (2)
+DIP40 3
+</text>
 </plain>
 <instances>
